File: pcb/cpu.sch (KiCad schematic (older format))
At the start: 2 parts, among them U100 MCIMX7S5EVM08SC

Commit message: pcb: working on sch
Parts:
- removed U?: MCIMX7S5EVM08SC, symbol symbols:MCIMX7S5EVM08SC
- added C100, C107, C108, C109: 220nF, symbol Device:C
- added C101, C102: 18pF-DNP, symbol Device:C
- added C103, C104: 18pF, symbol Device:C
- added C105, C106: 100nF, symbol Device:C
- added C110: 2.2uF, symbol Device:C
- added D100: 1N5819, symbol Device:D_Schottky
- added J100, J101: Conn_02x05_Odd_Even, symbol Connector_Generic:Conn_02x05_Odd_Even
- added J100: Conn_01x06, symbol Connector_Generic:Conn_01x06
- added R100: 100K, symbol Device:R
- added R101: 0, symbol Device:R
- added R102: 1M, symbol Device:R
- added R103: 4.75M-DNP, symbol Device:R
- added R104, R107: 10K-DNP, symbol Device:R
- added R105, R106, R108, R109, R110, R111: 10K, symbol Device:R
- added RN100, RN101, RN102: 10K, symbol Device:R_Pack04
- added unit 8 of U100
- added U?: Si5351A-B, symbol symbols:Si5351A-B
- added Y100: 24MHz, symbol Device:Crystal_GND24
- added Y101: 32.768kHz, symbol Device:Crystal
- added Y102: 25MHz, symbol Device:Crystal_GND24
Connections:
- net labels added: +1V8A, +3V3, BT_CFG_1, BT_CFG_10, BT_CFG_11, BT_CFG_12, BT_CFG_13, BT_CFG_14, BT_CFG_2, BT_CFG_3, BT_CFG_4, BT_CFG_5, BT_CFG_6, CPLD_JTAG_TCK, CPLD_JTAG_TDI, CPLD_JTAG_TDO, CPLD_JTAG_TMS, DAC_SYSCLK, GND, I2C1_SCL, I2C1_SDA, MPU_JTAG_TCK, MPU_JTAG_TDI, MPU_JTAG_TDO, MPU_JTAG_TMS, MPU_JTAG_TRST, PMIC_ON_REQ, PMIC_STBY_REQ, POR, SAI1_MCLK, UART3_CTS, UART3_RTS, UART3_RXD, UART3_TXD
- wire segments 0 -> 161
- no-connect marks 0 -> 18
Other:
- note added: "ARM JTAG"
- note added: "Audio PLL"
- note added: "BOOTMODE[1:0]:\n00 - Boot from fuses\n01 - Serial Downloader\n10 - Internal Boot\n11 - Reserved"
- note added: "CPLD JTAG"
- note added: "To WiFi & BT"
- moved on the sheet: U100B

Commit message: pcb: working on sch
Parts:
- removed C105, C106: 100nF, symbol Device:C
- removed U?: Si5351A-B, symbol symbols:Si5351A-B
- removed Y102: 25MHz, symbol Device:Crystal_GND24
Connections:
- net labels removed: DAC_SYSCLK, SAI1_MCLK
- wire segments 161 -> 143
- no-connect marks 18 -> 17
Other:
- note removed: "Audio PLL"
Changed lines of the file:
@@
 Wire Wire Line
 	4400 1950 3500 1950
-$Comp
-L symbols:Si5351A-B U?
-U 1 1 5D296AB4
-P 4700 6200
-F 0 "U?" H 4700 6865 50  0000 C CNN
-F 1 "Si5351A-B" H 4700 6774 50  0000 C CNN
-F 2 "" H 4700 6200 118 0001 C CNN
-F 3 "" H 4700 6200 118 0001 C CNN
-	1    4700 6200
-	1    0    0    -1
-$EndComp
-$Comp
-L Device:C C105
-U 1 1 5D298A03
-P 5400 6750
-F 0 "C105" H 5515 6796 50  0000 L CNN
-F 1 "100nF" H 5515 6705 50  0000 L CNN
-F 2 "" H 5438 6600 50  0001 C CNN
-F 3 "~" H 5400 6750 50  0001 C CNN
-	1    5400 6750
-	1    0    0    -1
-$EndComp
-$Comp
-L Device:C C106
-U 1 1 5D29A10C
-P 5800 6750
-F 0 "C106" H 5915 6796 50  0000 L CNN
-F 1 "100nF" H 5915 6705 50  0000 L CNN
-F 2 "" H 5838 6600 50  0001 C CNN
-F 3 "~" H 5800 6750 50  0001 C CNN
-	1    5800 6750
-	1    0    0    -1
-$EndComp
-$Comp
-L power:+3V3 #PWR?
-U 1 1 5D29ABDA
-P 5800 6400
-F 0 "#PWR?" H 5800 6250 50  0001 C CNN
-F 1 "+3V3" H 5815 6573 50  0000 C CNN
-F 2 "" H 5800 6400 50  0001 C CNN
-F 3 "" H 5800 6400 50  0001 C CNN
-	1    5800 6400
-	1    0    0    -1
-$EndComp
-Wire Wire Line
-	5300 6400 5400 6400
-Wire Wire Line
-	5800 6600 5800 6400
-Connection ~ 5800 6400
-Wire Wire Line
-	5300 6500 5400 6500
-Wire Wire Line
-	5400 6500 5400 6400
-Connection ~ 5400 6400
-Wire Wire Line
-	5400 6400 5800 6400
-Wire Wire Line
-	5400 6600 5400 6500
-Connection ~ 5400 6500
-$Comp
-L power:GND #PWR?
-U 1 1 5D2A787A
-P 5400 6900
-F 0 "#PWR?" H 5400 6650 50  0001 C CNN
-F 1 "GND" H 5405 6727 50  0000 C CNN
-F 2 "" H 5400 6900 50  0001 C CNN
-F 3 "" H 5400 6900 50  0001 C CNN
-	1    5400 6900
-	1    0    0    -1
-$EndComp
-$Comp
-L power:GND #PWR?
-U 1 1 5D2A7F4A
-P 5800 6900
-F 0 "#PWR?" H 5800 6650 50  0001 C CNN
-F 1 "GND" H 5805 6727 50  0000 C CNN
-F 2 "" H 5800 6900 50  0001 C CNN
-F 3 "" H 5800 6900 50  0001 C CNN
-	1    5800 6900
-	1    0    0    -1
-$EndComp
-$Comp
-L power:GND #PWR?
-U 1 1 5D2A8217
-P 4000 6950
-F 0 "#PWR?" H 4000 6700 50  0001 C CNN
-F 1 "GND" H 4005 6777 50  0000 C CNN
-F 2 "" H 4000 6950 50  0001 C CNN
-F 3 "" H 4000 6950 50  0001 C CNN
-	1    4000 6950
-	1    0    0    -1
-$EndComp
-Wire Wire Line
-	4100 6500 4000 6500
-Wire Wire Line
-	4000 6500 4000 6950
-$Comp
-L Device:Crystal_GND24 Y102
-U 1 1 5D2ABD38
-P 3700 5850
-F 0 "Y102" V 3500 5600 50  0000 L CNN
-F 1 "25MHz" V 3500 5900 50  0000 L CNN
-F 2 "" H 3700 5850 50  0001 C CNN
-F 3 "~" H 3700 5850 50  0001 C CNN
-	1    3700 5850
-	0    1    1    0
-$EndComp
-Wire Wire Line
-	4100 5700 3700 5700
-Wire Wire Line
-	4100 6000 3700 6000
-$Comp
-L power:GND #PWR?
-U 1 1 5D2BA4EB
-P 3500 6100
-F 0 "#PWR?" H 3500 5850 50  0001 C CNN
-F 1 "GND" V 3505 5972 50  0000 R CNN
-F 2 "" H 3500 6100 50  0001 C CNN
-F 3 "" H 3500 6100 50  0001 C CNN
-	1    3500 6100
-	0    1    1    0
-$EndComp
-Wire Wire Line
-	3500 5850 3500 6100
-Wire Wire Line
-	3900 5850 3900 6100
-Connection ~ 3500 6100
-Wire Wire Line
-	3500 6100 3900 6100
-Wire Wire Line
-	4100 5700 4100 5900
-Text GLabel 3850 6300 0    50   BiDi ~ 0
-I2C1_SDA
-Text GLabel 3850 6200 0    50   Input ~ 0
-I2C1_SCL
-Wire Wire Line
-	3850 6200 4100 6200
-Wire Wire Line
-	3850 6300 4100 6300
-Text GLabel 5500 6100 2    50   Output ~ 0
-DAC_SYSCLK
-Text GLabel 5500 5900 2    50   Output ~ 0
-SAI1_MCLK
-Wire Wire Line
-	5300 5900 5500 5900
-Wire Wire Line
-	5300 6100 5500 6100
-NoConn ~ 5300 6000
 Connection ~ 1700 5100
 $Comp
@@
 Wire Wire Line
 	8800 6100 8100 6100
-Text Notes 4400 5400 0    100  ~ 0
-Audio PLL
 Text Notes 8200 5500 0    100  ~ 0
 ARM JTAG

Commit message: pcb: finishing sch for r0.1
Parts:
- C100, C101, C102, C103, C104, C107, C108, C109, C110: footprint (none) -> Capacitor_SMD:C_0402_1005Metric
- D100: footprint (none) -> Diode_SMD:D_SOD-123
- J100, J101: footprint (none) -> Connector_PinHeader_1.27mm:PinHeader_2x05_P1.27mm_Vertical_SMD
- J100: value Conn_01x06 -> Conn_02x05_Odd_Even; footprint (none) -> Connector_PinHeader_1.27mm:PinHeader_2x05_P1.27mm_Vertical_SMD
- R100, R101, R102, R103, R104, R105, R106, R107, R108, R109, R110, R111: footprint (none) -> Resistor_SMD:R_0603_1608Metric
- RN100, RN101, RN102: footprint (none) -> Resistor_SMD:R_Array_Convex_4x0402
- U100: footprint (none) -> footprints:BGA-541_25x25_19.0x19.0mm
- Y100: footprint (none) -> Oscillator:Oscillator_SMD_Abracon_ASE-4Pin_3.2x2.5mm
- Y101: footprint (none) -> Crystal:Crystal_SMD_TXC_9HT11-2Pin_2.0x1.2mm_HandSoldering
Connections:
- net labels added: BAT_LOW, EXT_PWR_GOOD, PB_STAT, USB_SUSPEND
- wire segments 143 -> 147
- no-connect marks 17 -> 14

Commit message: pcb: initial netlist
Parts:
- renumbered J100 to J102
Changed lines of the file:
@@
 Connection ~ 8650 1400
 $Comp
-L Connector_Generic:Conn_01x06 J100
+L Connector_Generic:Conn_01x06 J102
 U 1 1 5DA9BBD7
 P 10200 3400
-F 0 "J100" H 10280 3392 50  0000 L CNN
+F 0 "J102" H 10280 3392 50  0000 L CNN
 F 1 "Conn_02x05_Odd_Even" H 10280 3301 50  0000 L CNN
 F 2 "Connector_PinHeader_1.27mm:PinHeader_2x05_P1.27mm_Vertical_SMD" H 10200 3400 50  0001 C CNN

Commit message: pcb: working on layout
Parts:
- removed R100: 100K, Resistor_SMD:R_0603_1608Metric, symbol Device:R
- removed R101: 0, Resistor_SMD:R_0603_1608Metric, symbol Device:R
Connections:
- wire segments 147 -> 145
Changed lines of the file:
@@
 Comment4 ""
 $EndDescr
-$Comp
-L symbols:MCIMX7S5EVM08SC U100
-U 2 1 5D4A59CF
-P 2700 3450
-F 0 "U100" H 2700 5815 50  0000 C CNN
-F 1 "MCIMX7S5EVM08SC" H 2700 5724 50  0000 C CNN
-F 2 "footprints:BGA-541_25x25_19.0x19.0mm" H 2700 4150 50  0001 C CNN
-F 3 "" H 2700 4150 50  0001 C CNN
-	2    2700 3450
-	1    0    0    -1
-$EndComp
 Text GLabel 1700 3350 0    50   Output ~ 0
 PMIC_STBY_REQ
@@
 	1700 1550 1900 1550
 $Comp
-L Device:R R100
-U 1 1 5D1AD784
-P 1650 2050
-F 0 "R100" V 1550 1900 50  0000 C CNN
-F 1 "100K" V 1550 2200 50  0000 C CNN
-F 2 "Resistor_SMD:R_0603_1608Metric" V 1580 2050 50  0001 C CNN
-F 3 "~" H 1650 2050 50  0001 C CNN
-	1    1650 2050
-	0    1    1    0
-$EndComp
-$Comp
 L power:GND #PWR0101
 U 1 1 5D1AEC8A
-P 1400 2050
-F 0 "#PWR0101" H 1400 1800 50  0001 C CNN
-F 1 "GND" H 1405 1877 50  0000 C CNN
-F 2 "" H 1400 2050 50  0001 C CNN
-F 3 "" H 1400 2050 50  0001 C CNN
-	1    1400 2050
+P 1800 2050
+F 0 "#PWR0101" H 1800 1800 50  0001 C CNN
+F 1 "GND" H 1805 1877 50  0000 C CNN
+F 2 "" H 1800 2050 50  0001 C CNN
+F 3 "" H 1800 2050 50  0001 C CNN
+	1    1800 2050
 	1    0    0    -1
 $EndComp
 Wire Wire Line
 	1900 2050 1800 2050
-Wire Wire Line
-	1500 2050 1400 2050
-$Comp
-L Device:R R101
-U 1 1 5D1B00E5
-P 3750 2950
-F 0 "R101" V 3650 2800 50  0000 C CNN
-F 1 "0" V 3650 3100 50  0000 C CNN
-F 2 "Resistor_SMD:R_0603_1608Metric" V 3680 2950 50  0001 C CNN
-F 3 "~" H 3750 2950 50  0001 C CNN
-	1    3750 2950
-	0    1    1    0
-$EndComp
 $Comp
 L power:GND #PWR0102
 U 1 1 5D1B0DA3
-P 4000 2950
-F 0 "#PWR0102" H 4000 2700 50  0001 C CNN
-F 1 "GND" H 4005 2777 50  0000 C CNN
-F 2 "" H 4000 2950 50  0001 C CNN
-F 3 "" H 4000 2950 50  0001 C CNN
-	1    4000 2950
-	1    0    0    -1
-$EndComp
-Wire Wire Line
-	3900 2950 4000 2950
-Wire Wire Line
-	3600 2950 3500 2950
+P 3600 2950
+F 0 "#PWR0102" H 3600 2700 50  0001 C CNN
+F 1 "GND" H 3605 2777 50  0000 C CNN
+F 2 "" H 3600 2950 50  0001 C CNN
+F 3 "" H 3600 2950 50  0001 C CNN
+	1    3600 2950
+	1    0    0    -1
+$EndComp
+Wire Wire Line
+	3500 2950 3600 2950
 NoConn ~ 3500 2650
 NoConn ~ 3500 2750
@@
 	2600 5900 2600 6900
 Wire Wire Line
-	2500 6100 2500 6900
-Wire Wire Line
-	1400 6100 2500 6100
-Wire Wire Line
-	2400 6200 2400 6900
-Wire Wire Line
-	1400 6200 2400 6200
-Wire Wire Line
 	2000 6300 2000 6900
 Wire Wire Line
 	1400 6300 2000 6300
 Wire Wire Line
-	1900 6400 1900 6900
-Wire Wire Line
-	1400 6400 1900 6400
-Wire Wire Line
 	1400 6500 1800 6500
 Wire Wire Line
@@
 Wire Wire Line
 	1800 6600 1800 6900
-Wire Wire Line
-	1400 6700 1700 6700
-Wire Wire Line
-	1700 6700 1700 6900
 $Comp
 L power:GND #PWR0107
@@
 Text GLabel 1700 3050 0    50   Input ~ 0
 PB_STAT
-Text GLabel 1700 2950 0    50   Input ~ 0
+Text GLabel 1250 3900 0    50   Input ~ 0
 EXT_PWR_GOOD
 Text GLabel 1700 3150 0    50   Input ~ 0
 BAT_LOW
-Text GLabel 1700 2850 0    50   Output ~ 0
+Text GLabel 1250 3800 0    50   Output ~ 0
 USB_SUSPEND
 Wire Wire Line
-	1700 2850 1900 2850
-Wire Wire Line
-	1700 2950 1900 2950
+	1250 3800 1450 3800
+Wire Wire Line
+	1250 3900 1450 3900
 Wire Wire Line
 	1700 3050 1900 3050
@@
 	1700 3150 1900 3150
 NoConn ~ 1900 1450
+$Comp
+L symbols:MCIMX7S5EVM08SC U100
+U 2 1 5D4A59CF
+P 2700 3450
+F 0 "U100" H 2700 5815 50  0000 C CNN
+F 1 "MCIMX7S5EVM08SC" H 2700 5724 50  0000 C CNN
+F 2 "footprints:BGA-541_25x25_19.0x19.0mm" H 2700 4150 50  0001 C CNN
+F 3 "" H 2700 4150 50  0001 C CNN
+	2    2700 3450
+	1    0    0    -1
+$EndComp
+Wire Wire Line
+	2500 6200 2500 6900
+Wire Wire Line
+	1400 6200 2500 6200
+Wire Wire Line
+	1400 6100 2400 6100
+Wire Wire Line
+	2400 6100 2400 6900
+Wire Wire Line
+	1900 6700 1900 6900
+Wire Wire Line
+	1400 6700 1900 6700
+Wire Wire Line
+	1400 6400 1700 6400
+Wire Wire Line
+	1700 6400 1700 6900
 $EndSCHEMATC

Commit message: pcb: add board outline
Parts:
- removed C109: 220nF, Capacitor_SMD:C_0402_1005Metric, symbol Device:C
Connections:
- wire segments 145 -> 143
- no-connect marks 14 -> 12
Other:
- note added: "There are already lot of decoupling\ncaps just next to it."
- moved on the sheet: R104, R105, R106, R107
Changed lines of the file:
@@
 NoConn ~ 3500 2350
-$Comp
-L symbols:+1V8A #PWR0103
-U 1 1 5D1B2FF0
-P 1800 3650
-F 0 "#PWR0103" H 1800 3500 50  0001 C CNN
-F 1 "+1V8A" H 1600 3700 50  0000 C CNN
-F 2 "" H 1800 3650 50  0001 C CNN
-F 3 "" H 1800 3650 50  0001 C CNN
-	1    1800 3650
-	1    0    0    -1
-$EndComp
 $Comp
 L Device:C C100
@@
 Wire Wire Line
 	1800 3750 1800 3650
-Connection ~ 1800 3650
 $Comp
 L power:GND #PWR0104
@@
 L Device:R R104
 U 1 1 5D2235B5
-P 1200 1500
-F 0 "R104" V 1100 1350 50  0000 C CNN
-F 1 "10K-DNP" V 1100 1650 50  0000 C CNN
-F 2 "Resistor_SMD:R_0603_1608Metric" V 1130 1500 50  0001 C CNN
-F 3 "~" H 1200 1500 50  0001 C CNN
-	1    1200 1500
-	-1   0    0    1
-$EndComp
-$Comp
-L Device:R R105
-U 1 1 5D2243E3
-P 1200 2100
-F 0 "R105" V 1100 1950 50  0000 C CNN
-F 1 "10K" V 1100 2250 50  0000 C CNN
-F 2 "Resistor_SMD:R_0603_1608Metric" V 1130 2100 50  0001 C CNN
-F 3 "~" H 1200 2100 50  0001 C CNN
-	1    1200 2100
-	-1   0    0    1
-$EndComp
-$Comp
-L Device:R R106
-U 1 1 5D225B1C
 P 1000 1500
-F 0 "R106" V 900 1350 50  0000 C CNN
-F 1 "10K" V 900 1650 50  0000 C CNN
+F 0 "R104" V 900 1350 50  0000 C CNN
+F 1 "10K-DNP" V 900 1650 50  0000 C CNN
 F 2 "Resistor_SMD:R_0603_1608Metric" V 930 1500 50  0001 C CNN
 F 3 "~" H 1000 1500 50  0001 C CNN
@@
 $EndComp
 $Comp
-L Device:R R107
-U 1 1 5D225B22
+L Device:R R105
+U 1 1 5D2243E3
 P 1000 2100
-F 0 "R107" V 900 1950 50  0000 C CNN
-F 1 "10K-DNP" V 900 2250 50  0000 C CNN
+F 0 "R105" V 900 1950 50  0000 C CNN
+F 1 "10K" V 900 2250 50  0000 C CNN
 F 2 "Resistor_SMD:R_0603_1608Metric" V 930 2100 50  0001 C CNN
 F 3 "~" H 1000 2100 50  0001 C CNN
@@
 $EndComp
 $Comp
+L Device:R R106
+U 1 1 5D225B1C
+P 800 1500
+F 0 "R106" V 700 1350 50  0000 C CNN
+F 1 "10K" V 700 1650 50  0000 C CNN
+F 2 "Resistor_SMD:R_0603_1608Metric" V 730 1500 50  0001 C CNN
+F 3 "~" H 800 1500 50  0001 C CNN
+	1    800  1500
+	-1   0    0    1
+$EndComp
+$Comp
+L Device:R R107
+U 1 1 5D225B22
+P 800 2100
+F 0 "R107" V 700 1950 50  0000 C CNN
+F 1 "10K-DNP" V 700 2250 50  0000 C CNN
+F 2 "Resistor_SMD:R_0603_1608Metric" V 730 2100 50  0001 C CNN
+F 3 "~" H 800 2100 50  0001 C CNN
+	1    800  2100
+	-1   0    0    1
+$EndComp
+$Comp
 L power:GND #PWR0109
 U 1 1 5D227422
-P 1200 2450
-F 0 "#PWR0109" H 1200 2200 50  0001 C CNN
-F 1 "GND" H 1205 2277 50  0000 C CNN
-F 2 "" H 1200 2450 50  0001 C CNN
-F 3 "" H 1200 2450 50  0001 C CNN
-	1    1200 2450
+P 1000 2450
+F 0 "#PWR0109" H 1000 2200 50  0001 C CNN
+F 1 "GND" H 1005 2277 50  0000 C CNN
+F 2 "" H 1000 2450 50  0001 C CNN
+F 3 "" H 1000 2450 50  0001 C CNN
+	1    1000 2450
 	1    0    0    -1
 $EndComp
@@
 L power:+3V3 #PWR0110
 U 1 1 5D2286DE
-P 1200 1150
-F 0 "#PWR0110" H 1200 1000 50  0001 C CNN
-F 1 "+3V3" H 1215 1323 50  0000 C CNN
-F 2 "" H 1200 1150 50  0001 C CNN
-F 3 "" H 1200 1150 50  0001 C CNN
-	1    1200 1150
-	1    0    0    -1
-$EndComp
-Wire Wire Line
-	1900 1750 1200 1750
-Wire Wire Line
-	1200 1750 1200 1950
-Wire Wire Line
-	1200 1650 1200 1750
-Connection ~ 1200 1750
-Wire Wire Line
-	1900 1850 1000 1850
-Wire Wire Line
-	1000 1850 1000 1950
-Wire Wire Line
-	1000 1650 1000 1850
-Connection ~ 1000 1850
+P 1000 1150
+F 0 "#PWR0110" H 1000 1000 50  0001 C CNN
+F 1 "+3V3" H 1015 1323 50  0000 C CNN
+F 2 "" H 1000 1150 50  0001 C CNN
+F 3 "" H 1000 1150 50  0001 C CNN
+	1    1000 1150
+	1    0    0    -1
+$EndComp
+Wire Wire Line
+	1000 1750 1000 1950
+Wire Wire Line
+	1000 1650 1000 1750
+Connection ~ 1000 1750
+Wire Wire Line
+	800  1850 800  1950
+Wire Wire Line
+	800  1650 800  1850
+Connection ~ 800  1850
+Wire Wire Line
+	800  1350 800  1150
+Wire Wire Line
+	800  1150 1000 1150
 Wire Wire Line
 	1000 1350 1000 1150
-Wire Wire Line
-	1000 1150 1200 1150
-Wire Wire Line
-	1200 1350 1200 1150
-Connection ~ 1200 1150
-Wire Wire Line
-	1200 2250 1200 2450
+Connection ~ 1000 1150
 Wire Wire Line
 	1000 2250 1000 2450
 Wire Wire Line
-	1000 2450 1200 2450
-Connection ~ 1200 2450
+	800  2250 800  2450
+Wire Wire Line
+	800  2450 1000 2450
+Connection ~ 1000 2450
 NoConn ~ 1900 2250
-NoConn ~ 1900 2350
-NoConn ~ 1900 2450
 NoConn ~ 1900 2550
 NoConn ~ 1900 2650
@@
 L power:+3V3 #PWR?
 U 1 1 5D9EC1DD
-P 6400 3500
+P 6600 3500
 AR Path="/5DB2122B/5D9EC1DD" Ref="#PWR?"  Part="1"
 AR Path="/5D180A01/5D9EC1DD" Ref="#PWR0120"  Part="1"
-F 0 "#PWR0120" H 6400 3350 50  0001 C CNN
-F 1 "+3V3" H 6415 3673 50  0000 C CNN
-F 2 "" H 6400 3500 50  0001 C CNN
-F 3 "" H 6400 3500 50  0001 C CNN
-	1    6400 3500
-	1    0    0    -1
-$EndComp
-$Comp
-L Device:C C?
-U 1 1 5D9EC1E3
-P 6400 3850
-AR Path="/5DB2122B/5D9EC1E3" Ref="C?"  Part="1"
-AR Path="/5D180A01/5D9EC1E3" Ref="C109"  Part="1"
-F 0 "C109" H 6515 3896 50  0000 L CNN
-F 1 "220nF" H 6515 3805 50  0000 L CNN
-F 2 "Capacitor_SMD:C_0402_1005Metric" H 6438 3700 50  0001 C CNN
-F 3 "~" H 6400 3850 50  0001 C CNN
-	1    6400 3850
-	1    0    0    -1
-$EndComp
-$Comp
-L power:GND #PWR?
-U 1 1 5D9EC1E9
-P 6400 4100
-AR Path="/5DB2122B/5D9EC1E9" Ref="#PWR?"  Part="1"
-AR Path="/5D180A01/5D9EC1E9" Ref="#PWR0121"  Part="1"
-F 0 "#PWR0121" H 6400 3850 50  0001 C CNN
-F 1 "GND" H 6405 3927 50  0000 C CNN
-F 2 "" H 6400 4100 50  0001 C CNN
-F 3 "" H 6400 4100 50  0001 C CNN
-	1    6400 4100
-	1    0    0    -1
-$EndComp
-Wire Wire Line
-	6400 3500 6400 3700
-Wire Wire Line
-	6400 4100 6400 4000
-Connection ~ 6400 3500
+F 0 "#PWR0120" H 6600 3350 50  0001 C CNN
+F 1 "+3V3" H 6615 3673 50  0000 C CNN
+F 2 "" H 6600 3500 50  0001 C CNN
+F 3 "" H 6600 3500 50  0001 C CNN
+	1    6600 3500
+	1    0    0    -1
+$EndComp
 $Comp
 L Device:C C?
@@
 	1    0    0    -1
 $EndComp
-Wire Wire Line
-	6400 3500 6800 3500
 Text GLabel 9500 1300 2    50   Output ~ 0
 I2C1_SCL
@@
 Text GLabel 1700 3050 0    50   Input ~ 0
 PB_STAT
-Text GLabel 1250 3900 0    50   Input ~ 0
+Text GLabel 1700 2450 0    50   Input ~ 0
 EXT_PWR_GOOD
 Text GLabel 1700 3150 0    50   Input ~ 0
 BAT_LOW
-Text GLabel 1250 3800 0    50   Output ~ 0
+Text GLabel 1700 2350 0    50   Output ~ 0
 USB_SUSPEND
 Wire Wire Line
-	1250 3800 1450 3800
-Wire Wire Line
-	1250 3900 1450 3900
+	1700 2350 1900 2350
+Wire Wire Line
+	1700 2450 1900 2450
 Wire Wire Line
 	1700 3050 1900 3050
@@
 Wire Wire Line
 	1700 6400 1700 6900
+Text Notes 5950 3700 0    50   ~ 0
+There are already lot of decoupling\ncaps just next to it.
+Wire Wire Line
+	6600 3500 6800 3500
+$Comp
+L symbols:+1V8A #PWR0103
+U 1 1 5D244741
+P 1800 3650
+F 0 "#PWR0103" H 1800 3500 50  0001 C CNN
+F 1 "+1V8A" H 1815 3823 50  0000 C CNN
+F 2 "" H 1800 3650 50  0001 C CNN
+F 3 "" H 1800 3650 50  0001 C CNN
+	1    1800 3650
+	1    0    0    -1
+$EndComp
+Connection ~ 1800 3650
+Wire Wire Line
+	1000 1750 1900 1750
+Wire Wire Line
+	800  1850 1900 1850
 $EndSCHEMATC
