File: pcb/cpu.sch (KiCad schematic (older format))
At the start: 28 parts, among them J100 Conn_02x05_Odd_Even, J101 Conn_02x05_Odd_Even, J102 Conn_02x05_Odd_Even, U100 MCIMX7S5EVM08SC, Y100 24MHz, Y101 32.768kHz

Commit message: pcb: routing
Parts:
- C100, C101, C102, C103, C104, C107, C108, C110: symbol Device:C -> pcb-rescue:C-Device
- D100: symbol Device:D_Schottky -> pcb-rescue:D_Schottky-Device
- J100, J101: symbol Connector_Generic:Conn_02x05_Odd_Even -> pcb-rescue:Conn_02x05_Odd_Even-Connector_Generic
- J102: footprint Connector_PinHeader_1.27mm:PinHeader_2x05_P1.27mm_Vertical_SMD -> Connector_PinHeader_1.27mm:PinHeader_1x06_P1.27mm_Vertical; symbol Connector_Generic:Conn_01x06 -> pcb-rescue:Conn_01x06-Connector_Generic
- R102, R103, R104, R105, R106, R107, R108, R109, R110, R111: symbol Device:R -> pcb-rescue:R-Device
- RN100, RN101, RN102: symbol Device:R_Pack04 -> pcb-rescue:R_Pack04-Device
- Y100: symbol Device:Crystal_GND24 -> pcb-rescue:Crystal_GND24-Device
- Y101: symbol Device:Crystal -> pcb-rescue:Crystal-Device
Connections:
- no-connect marks 12 -> 14
Changed lines of the file:
@@
 	1700 1550 1900 1550
 $Comp
-L power:GND #PWR0101
+L pcb-rescue:GND-power #PWR0101
 U 1 1 5D1AEC8A
 P 1800 2050
@@
 	1900 2050 1800 2050
 $Comp
-L power:GND #PWR0102
+L pcb-rescue:GND-power #PWR0102
 U 1 1 5D1B0DA3
 P 3600 2950
@@
 NoConn ~ 3500 2350
 $Comp
-L Device:C C100
+L pcb-rescue:C-Device C100
 U 1 1 5D1B3DE6
 P 1800 3900
@@
 	1800 3750 1800 3650
 $Comp
-L power:GND #PWR0104
+L pcb-rescue:GND-power #PWR0104
 U 1 1 5D1B612A
 P 1800 4150
@@
 	1800 4050 1800 4150
 $Comp
-L Device:Crystal Y101
+L pcb-rescue:Crystal-Device Y101
 U 1 1 5D1B84E0
 P 5250 3750
@@
 $EndComp
 $Comp
-L Device:Crystal_GND24 Y100
+L pcb-rescue:Crystal_GND24-Device Y100
 U 1 1 5D1BAE47
 P 4350 4050
@@
 $EndComp
 $Comp
-L Device:C C101
+L pcb-rescue:C-Device C101
 U 1 1 5D1BC145
 P 5000 4000
@@
 $EndComp
 $Comp
-L Device:C C102
+L pcb-rescue:C-Device C102
 U 1 1 5D1BD063
 P 5500 4000
@@
 $EndComp
 $Comp
-L power:GND #PWR0105
+L pcb-rescue:GND-power #PWR0105
 U 1 1 5D1BD44D
 P 5000 4150
@@
 $EndComp
 $Comp
-L Device:C C103
+L pcb-rescue:C-Device C103
 U 1 1 5D1C36A2
 P 4100 4300
@@
 $EndComp
 $Comp
-L Device:C C104
+L pcb-rescue:C-Device C104
 U 1 1 5D1C36A8
 P 4600 4300
@@
 $EndComp
 $Comp
-L power:GND #PWR0106
+L pcb-rescue:GND-power #PWR0106
 U 1 1 5D1C36AE
 P 4100 4450
@@
 $EndComp
 $Comp
-L Device:R R102
+L pcb-rescue:R-Device R102
 U 1 1 5D1C3964
 P 4350 3650
@@
 $EndComp
 $Comp
-L Device:R R103
+L pcb-rescue:R-Device R103
 U 1 1 5D1C4735
 P 5250 3350
@@
 BT_CFG_14
 $Comp
-L Device:R_Pack04 RN100
+L pcb-rescue:R_Pack04-Device RN100
 U 1 1 5D1FE095
 P 1900 7100
@@
 $EndComp
 $Comp
-L Device:R_Pack04 RN101
+L pcb-rescue:R_Pack04-Device RN101
 U 1 1 5D2005B7
 P 2600 7100
@@
 $EndComp
 $Comp
-L Device:R_Pack04 RN102
+L pcb-rescue:R_Pack04-Device RN102
 U 1 1 5D206895
 P 1900 5300
@@
 	1800 6600 1800 6900
 $Comp
-L power:GND #PWR0107
+L pcb-rescue:GND-power #PWR0107
 U 1 1 5D21E58A
 P 1700 7300
@@
 $EndComp
 $Comp
-L power:+3V3 #PWR0108
+L pcb-rescue:+3V3-power #PWR0108
 U 1 1 5D21F0D5
 P 1700 5100
@@
 	2600 7300 2500 7300
 $Comp
-L Device:R R104
+L pcb-rescue:R-Device R104
 U 1 1 5D2235B5
 P 1000 1500
@@
 $EndComp
 $Comp
-L Device:R R105
+L pcb-rescue:R-Device R105
 U 1 1 5D2243E3
 P 1000 2100
@@
 $EndComp
 $Comp
-L Device:R R106
+L pcb-rescue:R-Device R106
 U 1 1 5D225B1C
 P 800 1500
@@
 $EndComp
 $Comp
-L Device:R R107
+L pcb-rescue:R-Device R107
 U 1 1 5D225B22
 P 800 2100
@@
 $EndComp
 $Comp
-L power:GND #PWR0109
+L pcb-rescue:GND-power #PWR0109
 U 1 1 5D227422
 P 1000 2450
@@
 $EndComp
 $Comp
-L power:+3V3 #PWR0110
+L pcb-rescue:+3V3-power #PWR0110
 U 1 1 5D2286DE
 P 1000 1150
@@
 NoConn ~ 1900 2750
 $Comp
-L power:GND #PWR0111
+L pcb-rescue:GND-power #PWR0111
 U 1 1 5D258935
 P 3600 2050
@@
 Connection ~ 1700 5100
 $Comp
-L Connector_Generic:Conn_02x05_Odd_Even J100
+L pcb-rescue:Conn_02x05_Odd_Even-Connector_Generic J100
 U 1 1 5D31C612
 P 7300 5900
@@
 $EndComp
 $Comp
-L power:+3V3 #PWR0112
+L pcb-rescue:+3V3-power #PWR0112
 U 1 1 5D32043C
 P 7000 5200
@@
 $EndComp
 $Comp
-L Device:R R108
+L pcb-rescue:R-Device R108
 U 1 1 5D32601B
 P 7700 5350
@@
 $EndComp
 $Comp
-L Device:R R109
+L pcb-rescue:R-Device R109
 U 1 1 5D327514
 P 8000 5350
@@
 Connection ~ 7000 5200
 $Comp
-L power:GND #PWR0113
+L pcb-rescue:GND-power #PWR0113
 U 1 1 5D35B6F4
 P 7000 6200
@@
 NoConn ~ 7100 6000
 $Comp
-L Device:D_Schottky D100
+L pcb-rescue:D_Schottky-Device D100
 U 1 1 5D37EF0D
 P 7950 6100
@@
 	9100 5500 9100 5700
 $Comp
-L power:+3V3 #PWR0114
+L pcb-rescue:+3V3-power #PWR0114
 U 1 1 5D3BDEDA
 P 9100 5500
@@
 $EndComp
 $Comp
-L power:GND #PWR0115
+L pcb-rescue:GND-power #PWR0115
 U 1 1 5D3BDA94
 P 9100 6200
@@
 CPLD JTAG
 $Comp
-L Connector_Generic:Conn_02x05_Odd_Even J101
+L pcb-rescue:Conn_02x05_Odd_Even-Connector_Generic J101
 U 1 1 5D31F9CC
 P 9400 5900
@@
 $EndComp
 $Comp
-L power:+3V3 #PWR?
+L pcb-rescue:+3V3-power #PWR?
 U 1 1 5D9DFFB8
 P 6600 1300
@@
 $EndComp
 $Comp
-L Device:C C?
+L pcb-rescue:C-Device C?
 U 1 1 5D9DFFBE
 P 6600 1650
@@
 $EndComp
 $Comp
-L power:GND #PWR?
+L pcb-rescue:GND-power #PWR?
 U 1 1 5D9DFFC4
 P 6600 1900
@@
 Connection ~ 6600 1300
 $Comp
-L power:+3V3 #PWR?
+L pcb-rescue:+3V3-power #PWR?
 U 1 1 5D9E5D3F
 P 6600 2500
@@
 $EndComp
 $Comp
-L Device:C C?
+L pcb-rescue:C-Device C?
 U 1 1 5D9E5D45
 P 6600 2850
@@
 $EndComp
 $Comp
-L power:GND #PWR?
+L pcb-rescue:GND-power #PWR?
 U 1 1 5D9E5D4B
 P 6600 3100
@@
 Connection ~ 6600 2500
 $Comp
-L power:+3V3 #PWR?
+L pcb-rescue:+3V3-power #PWR?
 U 1 1 5D9EC1DD
 P 6600 3500
@@
 $EndComp
 $Comp
-L Device:C C?
+L pcb-rescue:C-Device C?
 U 1 1 5D9F4B12
 P 6600 4250
@@
 	6600 4000 6600 4100
 $Comp
-L power:GND #PWR0122
+L pcb-rescue:GND-power #PWR0122
 U 1 1 5D9F4B1A
 P 6600 4400
@@
 	8400 1400 8650 1400
 $Comp
-L Device:R R110
+L pcb-rescue:R-Device R110
 U 1 1 5DA710EB
 P 8650 1050
@@
 $EndComp
 $Comp
-L Device:R R111
+L pcb-rescue:R-Device R111
 U 1 1 5DA7199D
 P 9050 1050
@@
 	8650 1200 8650 1400
 $Comp
-L power:+3V3 #PWR?
+L pcb-rescue:+3V3-power #PWR?
 U 1 1 5DA800C1
 P 8650 900
@@
 Connection ~ 8650 1400
 $Comp
-L Connector_Generic:Conn_01x06 J102
+L pcb-rescue:Conn_01x06-Connector_Generic J102
 U 1 1 5DA9BBD7
 P 10200 3400
 F 0 "J102" H 10280 3392 50  0000 L CNN
 F 1 "Conn_02x05_Odd_Even" H 10280 3301 50  0000 L CNN
-F 2 "Connector_PinHeader_1.27mm:PinHeader_2x05_P1.27mm_Vertical_SMD" H 10200 3400 50  0001 C CNN
+F 2 "Connector_PinHeader_1.27mm:PinHeader_1x06_P1.27mm_Vertical" H 10200 3400 50  0001 C CNN
 F 3 "~" H 10200 3400 50  0001 C CNN
 	1    10200 3400
@@
 	8400 3600 10000 3600
 $Comp
-L power:GND #PWR0124
+L pcb-rescue:GND-power #PWR0124
 U 1 1 5DAAF59A
 P 9900 3300
@@
 Text Notes 11050 4300 2    100  ~ 0
 To WiFi & BT
-Text GLabel 1700 3050 0    50   Input ~ 0
+Text GLabel 1700 1450 0    50   Input ~ 0
 PB_STAT
 Text GLabel 1700 2450 0    50   Input ~ 0
@@
 	1700 2450 1900 2450
 Wire Wire Line
-	1700 3050 1900 3050
+	1700 1450 1900 1450
 Wire Wire Line
 	1700 3150 1900 3150
-NoConn ~ 1900 1450
+NoConn ~ 1900 3050
 $Comp
 L symbols:MCIMX7S5EVM08SC U100
@@
 Wire Wire Line
 	800  1850 1900 1850
+NoConn ~ 1900 2850
+NoConn ~ 1900 2950
 $EndSCHEMATC
