File: pcb/usb.sch (KiCad schematic (older format))
At the start: 19 parts, among them J600 USB_B_Micro, U100 MCIMX7S5EVM08SC, U600 USBLC6-2SC6

Commit message: pcb: routing
Parts:
- C600, C601, C602, C603, C604, C605, C606, C607: symbol Device:C -> pcb-rescue:C-Device
- D600, D601: symbol Device:D_TVS -> pcb-rescue:D_TVS-Device
- J600: symbol Connector:USB_B_Micro -> pcb-rescue:USB_B_Micro-Connector
- R600, R601, R602, R603, R605, R608: symbol Device:R -> pcb-rescue:R-Device
- U600: symbol Power_Protection:USBLC6-2SC6 -> pcb-rescue:USBLC6-2SC6-Power_Protection
Changed lines of the file:
@@
 $EndDescr
 $Comp
-L Connector:USB_B_Micro J600
+L pcb-rescue:USB_B_Micro-Connector J600
 U 1 1 5C995A78
 P 9000 3000
@@
 $EndComp
 $Comp
-L Power_Protection:USBLC6-2SC6 U600
+L pcb-rescue:USBLC6-2SC6-Power_Protection U600
 U 1 1 5C995C17
 P 7900 2000
@@
 $EndComp
 $Comp
-L Device:D_TVS D600
+L pcb-rescue:D_TVS-Device D600
 U 1 1 5C995D76
 P 8100 3550
@@
 $EndComp
 $Comp
-L Device:D_TVS D601
+L pcb-rescue:D_TVS-Device D601
 U 1 1 5C995E54
 P 7600 3550
@@
 $EndComp
 $Comp
-L Device:R R600
+L pcb-rescue:R-Device R600
 U 1 1 5C995E96
 P 9100 3750
@@
 $EndComp
 $Comp
-L Device:C C607
+L pcb-rescue:C-Device C607
 U 1 1 5C995EF6
 P 8800 3750
@@
 $EndComp
 $Comp
-L Device:R R601
+L pcb-rescue:R-Device R601
 U 1 1 5C995F63
 P 6850 3000
@@
 $EndComp
 $Comp
-L Device:R R602
+L pcb-rescue:R-Device R602
 U 1 1 5C996037
 P 6850 3100
@@
 $EndComp
 $Comp
-L Device:C C600
+L pcb-rescue:C-Device C600
 U 1 1 5C9960AD
 P 5900 2150
@@
 $EndComp
 $Comp
-L power:GND #PWR0291
+L pcb-rescue:GND-power #PWR0291
 U 1 1 5C9961F9
 P 7900 2500
@@
 $EndComp
 $Comp
-L power:GND #PWR0292
+L pcb-rescue:GND-power #PWR0292
 U 1 1 5C996234
 P 9100 4100
@@
 $EndComp
 $Comp
-L power:GND #PWR0293
+L pcb-rescue:GND-power #PWR0293
 U 1 1 5C996258
 P 8100 3900
@@
 $EndComp
 $Comp
-L power:GND #PWR0294
+L pcb-rescue:GND-power #PWR0294
 U 1 1 5C99627A
 P 5900 2600
@@
 $EndComp
 $Comp
-L power:VBUS #PWR0295
+L pcb-rescue:VBUS-power #PWR0295
 U 1 1 5C9962B3
 P 5900 1900
@@
 Connection ~ 7200 2800
 $Comp
-L Device:R R603
+L pcb-rescue:R-Device R603
 U 1 1 5D1E0F87
 P 5650 3700
@@
 $EndComp
 $Comp
-L power:GND #PWR0296
+L pcb-rescue:GND-power #PWR0296
 U 1 1 5D1E2A0C
 P 6100 3700
@@
 	5300 3700 5500 3700
 $Comp
-L Device:R R605
+L pcb-rescue:R-Device R605
 U 1 1 5D1E8958
 P 5650 3600
@@
 $EndComp
 $Comp
-L power:+3V3 #PWR0298
+L pcb-rescue:+3V3-power #PWR0298
 U 1 1 5D1E9321
 P 6100 3600
@@
 NoConn ~ 5300 4800
 $Comp
-L power:+3V3 #PWR0299
+L pcb-rescue:+3V3-power #PWR0299
 U 1 1 5D20C9B4
 P 2500 3200
@@
 $EndComp
 $Comp
-L Device:C C?
+L pcb-rescue:C-Device C?
 U 1 1 5D2271CE
 P 2900 3650
@@
 $EndComp
 $Comp
-L Device:C C?
+L pcb-rescue:C-Device C?
 U 1 1 5D2271D4
 P 3300 3650
@@
 	3300 3500 3700 3500
 $Comp
-L power:GND #PWR?
+L pcb-rescue:GND-power #PWR?
 U 1 1 5D2271E4
 P 2900 3800
@@
 	3300 3800 2900 3800
 $Comp
-L Device:C C?
+L pcb-rescue:C-Device C?
 U 1 1 5D229E9F
 P 2500 3350
@@
 $EndComp
 $Comp
-L power:GND #PWR?
+L pcb-rescue:GND-power #PWR?
 U 1 1 5D22AF19
 P 2500 3500
@@
 Connection ~ 2500 3200
 $Comp
-L power:+3V3 #PWR0302
+L pcb-rescue:+3V3-power #PWR0302
 U 1 1 5D22EAC8
 P 2500 4100
@@
 $EndComp
 $Comp
-L Device:C C?
+L pcb-rescue:C-Device C?
 U 1 1 5D22EACE
 P 2900 4550
@@
 $EndComp
 $Comp
-L Device:C C?
+L pcb-rescue:C-Device C?
 U 1 1 5D22EAD4
 P 3300 4550
@@
 	3300 4400 3700 4400
 $Comp
-L power:GND #PWR?
+L pcb-rescue:GND-power #PWR?
 U 1 1 5D22EADD
 P 2900 4700
@@
 	3300 4700 2900 4700
 $Comp
-L Device:C C?
+L pcb-rescue:C-Device C?
 U 1 1 5D22EAE5
 P 2500 4250
@@
 $EndComp
 $Comp
-L power:GND #PWR?
+L pcb-rescue:GND-power #PWR?
 U 1 1 5D22EAEB
 P 2500 4400
@@
 The Type A port is not ESD protected, and only powered if Type B Micro is connected (shared power). \nThis port is meant for development purpose only.
 $Comp
-L Device:R R608
+L pcb-rescue:R-Device R608
 U 1 1 5D2D5A0B
 P 5900 2450
