File: pcb/usb.sch (KiCad schematic (older format))
At the start: 19 parts, among them J600 USB_B_Micro, U100 MCIMX7S5EVM08SC, U600 USBLC6-2SC6

Commit message: pcb: remap schematic symbols
Parts:
- C600, C601, C602, C603, C604, C605, C606, C607: symbol pcb-rescue:C-Device-pcb-rescue -> Device:C
- D600, D601: symbol pcb-rescue:D_TVS-Device-pcb-rescue -> Device:D_TVS
- J600: symbol pcb-rescue:USB_B_Micro-Connector-pcb-rescue -> Connector:USB_B_Micro
- R600, R601, R602, R603, R605, R608: symbol pcb-rescue:R-Device-pcb-rescue -> Device:R
- U600: symbol pcb-rescue:USBLC6-2SC6-Power_Protection-pcb-rescue -> Power_Protection:USBLC6-2SC6
Changed lines of the file:
@@
 $EndDescr
 $Comp
-L pcb-rescue:USB_B_Micro-Connector-pcb-rescue J600
+L Connector:USB_B_Micro J600
 U 1 1 5C995A78
 P 9000 3000
@@
 $EndComp
 $Comp
-L pcb-rescue:USBLC6-2SC6-Power_Protection-pcb-rescue U600
+L Power_Protection:USBLC6-2SC6 U600
 U 1 1 5C995C17
 P 7900 2000
@@
 $EndComp
 $Comp
-L pcb-rescue:D_TVS-Device-pcb-rescue D600
+L Device:D_TVS D600
 U 1 1 5C995D76
 P 8100 3550
@@
 $EndComp
 $Comp
-L pcb-rescue:D_TVS-Device-pcb-rescue D601
+L Device:D_TVS D601
 U 1 1 5C995E54
 P 7600 3550
@@
 $EndComp
 $Comp
-L pcb-rescue:R-Device-pcb-rescue R600
+L Device:R R600
 U 1 1 5C995E96
 P 9100 3750
@@
 $EndComp
 $Comp
-L pcb-rescue:C-Device-pcb-rescue C607
+L Device:C C607
 U 1 1 5C995EF6
 P 8800 3750
@@
 $EndComp
 $Comp
-L pcb-rescue:R-Device-pcb-rescue R601
+L Device:R R601
 U 1 1 5C995F63
 P 6850 3000
@@
 $EndComp
 $Comp
-L pcb-rescue:R-Device-pcb-rescue R602
+L Device:R R602
 U 1 1 5C996037
 P 6850 3100
@@
 $EndComp
 $Comp
-L pcb-rescue:C-Device-pcb-rescue C600
+L Device:C C600
 U 1 1 5C9960AD
 P 5900 2150
@@
 $EndComp
 $Comp
-L pcb-rescue:GND-power-pcb-rescue #PWR0291
+L power:GND #PWR0291
 U 1 1 5C9961F9
 P 7900 2500
@@
 $EndComp
 $Comp
-L pcb-rescue:GND-power-pcb-rescue #PWR0292
+L power:GND #PWR0292
 U 1 1 5C996234
 P 9100 4100
@@
 $EndComp
 $Comp
-L pcb-rescue:GND-power-pcb-rescue #PWR0293
+L power:GND #PWR0293
 U 1 1 5C996258
 P 8100 3900
@@
 $EndComp
 $Comp
-L pcb-rescue:GND-power-pcb-rescue #PWR0294
+L power:GND #PWR0294
 U 1 1 5C99627A
 P 5900 2600
@@
 $EndComp
 $Comp
-L pcb-rescue:VBUS-power-pcb-rescue #PWR0295
+L power:VBUS #PWR0295
 U 1 1 5C9962B3
 P 5900 1900
@@
 Connection ~ 7200 2800
 $Comp
-L pcb-rescue:R-Device-pcb-rescue R603
+L Device:R R603
 U 1 1 5D1E0F87
 P 5650 3700
@@
 $EndComp
 $Comp
-L pcb-rescue:GND-power-pcb-rescue #PWR0296
+L power:GND #PWR0296
 U 1 1 5D1E2A0C
 P 6100 3700
@@
 	5300 3700 5500 3700
 $Comp
-L pcb-rescue:R-Device-pcb-rescue R605
+L Device:R R605
 U 1 1 5D1E8958
 P 5650 3600
@@
 $EndComp
 $Comp
-L pcb-rescue:+3V3-power-pcb-rescue #PWR0298
+L power:+3V3 #PWR0298
 U 1 1 5D1E9321
 P 6100 3600
@@
 NoConn ~ 5300 4800
 $Comp
-L pcb-rescue:+3V3-power-pcb-rescue #PWR0299
+L power:+3V3 #PWR0299
 U 1 1 5D20C9B4
 P 2500 3200
@@
 $EndComp
 $Comp
-L pcb-rescue:C-Device-pcb-rescue C?
+L Device:C C?
 U 1 1 5D2271CE
 P 2900 3650
@@
 $EndComp
 $Comp
-L pcb-rescue:C-Device-pcb-rescue C?
+L Device:C C?
 U 1 1 5D2271D4
 P 3300 3650
@@
 	3300 3500 3700 3500
 $Comp
-L pcb-rescue:GND-power-pcb-rescue #PWR?
+L power:GND #PWR?
 U 1 1 5D2271E4
 P 2900 3800
@@
 	3300 3800 2900 3800
 $Comp
-L pcb-rescue:C-Device-pcb-rescue C?
+L Device:C C?
 U 1 1 5D229E9F
 P 2500 3350
@@
 $EndComp
 $Comp
-L pcb-rescue:GND-power-pcb-rescue #PWR?
+L power:GND #PWR?
 U 1 1 5D22AF19
 P 2500 3500
@@
 Connection ~ 2500 3200
 $Comp
-L pcb-rescue:+3V3-power-pcb-rescue #PWR0302
+L power:+3V3 #PWR0302
 U 1 1 5D22EAC8
 P 2500 4100
@@
 $EndComp
 $Comp
-L pcb-rescue:C-Device-pcb-rescue C?
+L Device:C C?
 U 1 1 5D22EACE
 P 2900 4550
@@
 $EndComp
 $Comp
-L pcb-rescue:C-Device-pcb-rescue C?
+L Device:C C?
 U 1 1 5D22EAD4
 P 3300 4550
@@
 	3300 4400 3700 4400
 $Comp
-L pcb-rescue:GND-power-pcb-rescue #PWR?
+L power:GND #PWR?
 U 1 1 5D22EADD
 P 2900 4700
@@
 	3300 4700 2900 4700
 $Comp
-L pcb-rescue:C-Device-pcb-rescue C?
+L Device:C C?
 U 1 1 5D22EAE5
 P 2500 4250
@@
 $EndComp
 $Comp
-L pcb-rescue:GND-power-pcb-rescue #PWR?
+L power:GND #PWR?
 U 1 1 5D22EAEB
 P 2500 4400
@@
 The Type A port is not ESD protected, and only powered if Type B Micro is connected (shared power). \nThis port is meant for development purpose only.
 $Comp
-L pcb-rescue:R-Device-pcb-rescue R608
+L Device:R R608
 U 1 1 5D2D5A0B
 P 5900 2450

Commit message: fix #2
Parts:
- removed R605: 47K, Resistor_SMD:R_0603_1608Metric, symbol Device:R
Connections:
- no-connect marks 8 -> 9
Other:
- note added: "The second USB is not present on iMX7 Solo.\n(But the second USB LDO does present)"
- note removed: "The second USB is not present on iMX7 Solo."
Changed lines of the file:
@@
 Wire Wire Line
 	5300 3700 5500 3700
-$Comp
-L Device:R R605
-U 1 1 5D1E8958
-P 5650 3600
-F 0 "R605" V 5600 3850 50  0000 C CNN
-F 1 "47K" V 5600 3300 50  0000 C CNN
-F 2 "Resistor_SMD:R_0603_1608Metric" V 5580 3600 50  0001 C CNN
-F 3 "~" H 5650 3600 50  0001 C CNN
-	1    5650 3600
-	0    -1   1    0
-$EndComp
-$Comp
-L power:+3V3 #PWR0298
-U 1 1 5D1E9321
-P 6100 3600
-F 0 "#PWR0298" H 6100 3450 50  0001 C CNN
-F 1 "+3V3" H 6100 3750 50  0000 C CNN
-F 2 "" H 6100 3600 50  0001 C CNN
-F 3 "" H 6100 3600 50  0001 C CNN
-	1    6100 3600
-	1    0    0    -1
-$EndComp
-Wire Wire Line
-	5800 3600 6100 3600
 Wire Wire Line
 	5800 3700 6100 3700
-Wire Wire Line
-	5500 3600 5300 3600
 NoConn ~ 5300 4700
 NoConn ~ 5300 4800
@@
 NoConn ~ 5300 4500
 Text Notes 5400 4300 0    50   ~ 0
-The second USB is not present on iMX7 Solo.
+The second USB is not present on iMX7 Solo.\n(But the second USB LDO does present)
+NoConn ~ 5300 3600
 $EndSCHEMATC
