File: pcb/ddr.sch (KiCad schematic (older format))
At the start: 36 parts, among them U100 MCIMX7S5EVM08SC, U200 IS43LD16128B

Commit message: pcb: rev 0.1
Parts:
- C200, C201, C202, C203, C204, C205, C206, C207, C208, C209, C210, C211, C212, C213, C214, C215, C216, C217, C218, C219, C220, C221, C222, C223, C224, C225, C226, C227: symbol pcb-rescue:C-Device -> pcb-rescue:C-Device-pcb-rescue
- L200: symbol pcb-rescue:L-Device -> pcb-rescue:L-Device-pcb-rescue
- R200, R201, R202, R203, R204: symbol pcb-rescue:R-Device -> pcb-rescue:R-Device-pcb-rescue
Changed lines of the file:
@@
 encoding utf-8
 Sheet 4 11
-Title "LPDDR2 SDRAM"
-Date ""
+Title "RhythmPocket"
+Date "2019-07-16"
 Rev "R0.1"
 Comp "ZephRay"
@@
 NoConn ~ 4500 5800
 $Comp
-L pcb-rescue:+1V2-power #PWR0171
+L pcb-rescue:+1V2-power-pcb-rescue #PWR0171
 U 1 1 5D6BF120
 P 6700 4800
@@
 $EndComp
 $Comp
-L pcb-rescue:+1V8-power #PWR0173
+L pcb-rescue:+1V8-power-pcb-rescue #PWR0173
 U 1 1 5D70B95B
 P 5750 5000
@@
 	6700 5100 6700 5000
 $Comp
-L pcb-rescue:L-Device L200
+L pcb-rescue:L-Device-pcb-rescue L200
 U 1 1 5D753562
 P 6100 5000
@@
 	6450 5200 6450 5000
 $Comp
-L pcb-rescue:GND-power #PWR0175
+L pcb-rescue:GND-power-pcb-rescue #PWR0175
 U 1 1 5D774EFD
 P 6800 6200
@@
 $EndComp
 $Comp
-L pcb-rescue:GND-power #PWR0176
+L pcb-rescue:GND-power-pcb-rescue #PWR0176
 U 1 1 5D77587F
 P 8200 6200
@@
 $EndComp
 $Comp
-L pcb-rescue:+1V2-power #PWR0177
+L pcb-rescue:+1V2-power-pcb-rescue #PWR0177
 U 1 1 5D77603C
 P 8300 4800
@@
 	8200 5800 8200 5700
 $Comp
-L pcb-rescue:R-Device R200
+L pcb-rescue:R-Device-pcb-rescue R200
 U 1 1 5D82DF01
 P 8450 4600
@@
 $EndComp
 $Comp
-L pcb-rescue:GND-power #PWR0178
+L pcb-rescue:GND-power-pcb-rescue #PWR0178
 U 1 1 5D82FD6C
 P 8800 4600
@@
 	8600 4600 8800 4600
 $Comp
-L pcb-rescue:R-Device R201
+L pcb-rescue:R-Device-pcb-rescue R201
 U 1 1 5D84AC72
 P 4850 7100
@@
 $EndComp
 $Comp
-L pcb-rescue:+1V2-power #PWR0180
+L pcb-rescue:+1V2-power-pcb-rescue #PWR0180
 U 1 1 5D84C76E
 P 6000 6500
@@
 $EndComp
 $Comp
-L pcb-rescue:GND-power #PWR0181
+L pcb-rescue:GND-power-pcb-rescue #PWR0181
 U 1 1 5D84E07D
 P 5200 7200
@@
 $EndComp
 $Comp
-L pcb-rescue:C-Device C200
+L pcb-rescue:C-Device-pcb-rescue C200
 U 1 1 5D84EB60
 P 5600 7050
@@
 $EndComp
 $Comp
-L pcb-rescue:C-Device C201
+L pcb-rescue:C-Device-pcb-rescue C201
 U 1 1 5D84F753
 P 6000 6750
@@
 $EndComp
 $Comp
-L pcb-rescue:GND-power #PWR0182
+L pcb-rescue:GND-power-pcb-rescue #PWR0182
 U 1 1 5D8503EC
 P 5600 7300
@@
 $EndComp
 $Comp
-L pcb-rescue:GND-power #PWR0183
+L pcb-rescue:GND-power-pcb-rescue #PWR0183
 U 1 1 5D8505EC
 P 6000 7000
@@
 	4500 6800 5600 6800
 $Comp
-L pcb-rescue:C-Device C202
+L pcb-rescue:C-Device-pcb-rescue C202
 U 1 1 5D8EF254
 P 800 6250
@@
 $EndComp
 $Comp
-L pcb-rescue:C-Device C203
+L pcb-rescue:C-Device-pcb-rescue C203
 U 1 1 5D8F02C4
 P 1200 6250
@@
 $EndComp
 $Comp
-L pcb-rescue:C-Device C204
+L pcb-rescue:C-Device-pcb-rescue C204
 U 1 1 5D8F075C
 P 1600 6250
@@
 $EndComp
 $Comp
-L pcb-rescue:C-Device C205
+L pcb-rescue:C-Device-pcb-rescue C205
 U 1 1 5D8F0A94
 P 2000 6250
@@
 $EndComp
 $Comp
-L pcb-rescue:C-Device C206
+L pcb-rescue:C-Device-pcb-rescue C206
 U 1 1 5D946198
 P 2400 6250
@@
 $EndComp
 $Comp
-L pcb-rescue:+1V2-power #PWR0184
+L pcb-rescue:+1V2-power-pcb-rescue #PWR0184
 U 1 1 5D947219
 P 800 6100
@@
 	2800 7000 2800 6900
 $Comp
-L pcb-rescue:GND-power #PWR0185
+L pcb-rescue:GND-power-pcb-rescue #PWR0185
 U 1 1 5DA15A1B
 P 800 6400
@@
 	2000 6400 1600 6400
 $Comp
-L pcb-rescue:C-Device C207
+L pcb-rescue:C-Device-pcb-rescue C207
 U 1 1 5DA309FE
 P 9200 1300
@@
 $EndComp
 $Comp
-L pcb-rescue:C-Device C208
+L pcb-rescue:C-Device-pcb-rescue C208
 U 1 1 5DA30A04
 P 9600 1300
@@
 $EndComp
 $Comp
-L pcb-rescue:C-Device C209
+L pcb-rescue:C-Device-pcb-rescue C209
 U 1 1 5DA30A16
 P 10000 1300
@@
 $EndComp
 $Comp
-L pcb-rescue:GND-power #PWR0186
+L pcb-rescue:GND-power-pcb-rescue #PWR0186
 U 1 1 5DA30A1C
 P 9200 1450
@@
 CAP for LPDDR_VDD2
 $Comp
-L pcb-rescue:C-Device C210
+L pcb-rescue:C-Device-pcb-rescue C210
 U 1 1 5DA70FA0
 P 9200 2200
@@
 $EndComp
 $Comp
-L pcb-rescue:C-Device C211
+L pcb-rescue:C-Device-pcb-rescue C211
 U 1 1 5DA70FA6
 P 9600 2200
@@
 $EndComp
 $Comp
-L pcb-rescue:C-Device C212
+L pcb-rescue:C-Device-pcb-rescue C212
 U 1 1 5DA70FAC
 P 10000 2200
@@
 $EndComp
 $Comp
-L pcb-rescue:C-Device C213
+L pcb-rescue:C-Device-pcb-rescue C213
 U 1 1 5DA70FB2
 P 10400 2200
@@
 $EndComp
 $Comp
-L pcb-rescue:C-Device C214
+L pcb-rescue:C-Device-pcb-rescue C214
 U 1 1 5DA70FB8
 P 10800 2200
@@
 $EndComp
 $Comp
-L pcb-rescue:GND-power #PWR0188
+L pcb-rescue:GND-power-pcb-rescue #PWR0188
 U 1 1 5DA70FBE
 P 9200 2350
@@
 	10400 2050 10000 2050
 $Comp
-L pcb-rescue:+1V2-power #PWR0189
+L pcb-rescue:+1V2-power-pcb-rescue #PWR0189
 U 1 1 5DA86AA7
 P 9200 2050
@@
 Connection ~ 9200 2050
 $Comp
-L pcb-rescue:C-Device C215
+L pcb-rescue:C-Device-pcb-rescue C215
 U 1 1 5DA8B14B
 P 9200 3100
@@
 $EndComp
 $Comp
-L pcb-rescue:C-Device C216
+L pcb-rescue:C-Device-pcb-rescue C216
 U 1 1 5DA8B151
 P 9600 3100
@@
 $EndComp
 $Comp
-L pcb-rescue:C-Device C217
+L pcb-rescue:C-Device-pcb-rescue C217
 U 1 1 5DA8B157
 P 10000 3100
@@
 $EndComp
 $Comp
-L pcb-rescue:C-Device C218
+L pcb-rescue:C-Device-pcb-rescue C218
 U 1 1 5DA8B15D
 P 10400 3100
@@
 $EndComp
 $Comp
-L pcb-rescue:C-Device C219
+L pcb-rescue:C-Device-pcb-rescue C219
 U 1 1 5DA8B163
 P 10800 3100
@@
 $EndComp
 $Comp
-L pcb-rescue:GND-power #PWR0190
+L pcb-rescue:GND-power-pcb-rescue #PWR0190
 U 1 1 5DA8B169
 P 9200 3250
@@
 	10400 2950 10000 2950
 $Comp
-L pcb-rescue:+1V2-power #PWR0191
+L pcb-rescue:+1V2-power-pcb-rescue #PWR0191
 U 1 1 5DA8B17E
 P 9200 2950
@@
 CAP for VDDQ
 $Comp
-L pcb-rescue:C-Device C220
+L pcb-rescue:C-Device-pcb-rescue C220
 U 1 1 5DAA272C
 P 9200 3850
@@
 $EndComp
 $Comp
-L pcb-rescue:C-Device C221
+L pcb-rescue:C-Device-pcb-rescue C221
 U 1 1 5DAA2732
 P 9600 3850
@@
 $EndComp
 $Comp
-L pcb-rescue:GND-power #PWR0192
+L pcb-rescue:GND-power-pcb-rescue #PWR0192
 U 1 1 5DAA2738
 P 9200 4000
@@
 	9600 4000 9200 4000
 $Comp
-L pcb-rescue:+1V2-power #PWR0193
+L pcb-rescue:+1V2-power-pcb-rescue #PWR0193
 U 1 1 5DAA2744
 P 9200 3700
@@
 	9600 1450 10000 1450
 $Comp
-L pcb-rescue:C-Device C222
+L pcb-rescue:C-Device-pcb-rescue C222
 U 1 1 5DAD61D9
 P 9200 4700
@@
 $EndComp
 $Comp
-L pcb-rescue:C-Device C223
+L pcb-rescue:C-Device-pcb-rescue C223
 U 1 1 5DAD61DF
 P 9600 4700
@@
 $EndComp
 $Comp
-L pcb-rescue:C-Device C224
+L pcb-rescue:C-Device-pcb-rescue C224
 U 1 1 5DAD61E5
 P 10000 4700
@@
 $EndComp
 $Comp
-L pcb-rescue:GND-power #PWR0194
+L pcb-rescue:GND-power-pcb-rescue #PWR0194
 U 1 1 5DAD61EB
 P 9200 4850
@@
 	9600 4850 10000 4850
 $Comp
-L pcb-rescue:+1V2-power #PWR0195
+L pcb-rescue:+1V2-power-pcb-rescue #PWR0195
 U 1 1 5DAEC398
 P 9200 4550
@@
 Connection ~ 9200 4550
 $Comp
-L pcb-rescue:C-Device C227
+L pcb-rescue:C-Device-pcb-rescue C227
 U 1 1 5DBFDA85
 P 9200 5750
@@
 $EndComp
 $Comp
-L pcb-rescue:C-Device C225
+L pcb-rescue:C-Device-pcb-rescue C225
 U 1 1 5DBFDE8B
 P 10200 5550
@@
 $EndComp
 $Comp
-L pcb-rescue:C-Device C226
+L pcb-rescue:C-Device-pcb-rescue C226
 U 1 1 5DBFE3CA
 P 10200 6050
@@
 $EndComp
 $Comp
-L pcb-rescue:R-Device R202
+L pcb-rescue:R-Device-pcb-rescue R202
 U 1 1 5DBFEB6C
 P 9600 5550
@@
 $EndComp
 $Comp
-L pcb-rescue:R-Device R203
+L pcb-rescue:R-Device-pcb-rescue R203
 U 1 1 5DBFF768
 P 9600 6050
@@
 $EndComp
 $Comp
-L pcb-rescue:GND-power #PWR0197
+L pcb-rescue:GND-power-pcb-rescue #PWR0197
 U 1 1 5DC70EC8
 P 9200 6200
@@
 $EndComp
 $Comp
-L pcb-rescue:+1V2-power #PWR0198
+L pcb-rescue:+1V2-power-pcb-rescue #PWR0198
 U 1 1 5DC711F6
 P 9200 5400
@@
 For LPDDR2,\nDRAM_RESET should be left unconnected\n
 $Comp
-L pcb-rescue:R-Device R204
+L pcb-rescue:R-Device-pcb-rescue R204
 U 1 1 5D1B9D3D
 P 4900 5250
@@
 	4900 5100 4900 5000
 $Comp
-L pcb-rescue:GND-power #PWR0199
+L pcb-rescue:GND-power-pcb-rescue #PWR0199
 U 1 1 5D1D2EB6
 P 4900 5400
