File: pcb/keypad.sch (KiCad schematic (older format))
At the start: 1 part

Commit message: pcb: finishing sch for r0.1
Parts:
- added C700, C701, C702: 220nF, Capacitor_SMD:C_0402_1005Metric, symbol Device:C
- added C703: 2.2uF, Capacitor_SMD:C_0402_1005Metric, symbol Device:C
- added L700: 120R, Inductor_SMD:L_0603_1608Metric, symbol Device:L
- added R700: 100K/1%, Resistor_SMD:R_0603_1608Metric, symbol Device:R
- added SW700, SW701, SW702, SW703, SW704, SW705, SW706, SW707: SW_Push, footprints:contact, symbol Switch:SW_Push
- added unit 10 of U100
- U100: renamed from U?; footprint (none) -> footprints:BGA-541_25x25_19.0x19.0mm
Connections:
- net labels added: +1V8, ADC1_IN0, ADC1_IN1, AP_WAKE_BT, BT_RST_N, BT_WAKE_AP, GND, SW_A, SW_B, SW_DN, SW_LE, SW_RI, SW_SE, SW_ST, SW_UP, WL_PMU_EN, WL_WAKE_AP, ~LCD_PWR_EN, ~SD_PWR_EN
- wire segments 1 -> 49
- no-connect marks 0 -> 3

Commit message: pcb: working on layout
Parts:
- removed C701: 220nF, Capacitor_SMD:C_0402_1005Metric, symbol Device:C
Connections:
- wire segments 49 -> 31
Other:
- moved on the sheet: C700, L700, SW702, SW703
Changed lines of the file:
@@
-$EndComp
-$Comp
-L Device:C C701
-U 1 1 5D256786
-P 6400 3350
-F 0 "C701" H 6515 3396 50  0000 L CNN
-F 1 "220nF" H 6515 3305 50  0000 L CNN
-F 2 "Capacitor_SMD:C_0402_1005Metric" H 6438 3200 50  0001 C CNN
-F 3 "~" H 6400 3350 50  0001 C CNN
-	1    6400 3350
-	1    0    0    -1
 $EndComp
 $Comp
@@
 	1    0    0    -1
 $EndComp
-$Comp
-L Device:L L700
-U 1 1 5D259B1C
-P 6150 3200
-F 0 "L700" V 6340 3200 50  0000 C CNN
-F 1 "120R" V 6249 3200 50  0000 C CNN
-F 2 "Inductor_SMD:L_0603_1608Metric" H 6150 3200 50  0001 C CNN
-F 3 "~" H 6150 3200 50  0001 C CNN
-	1    6150 3200
-	0    -1   -1   0
-$EndComp
-$Comp
-L Device:C C700
-U 1 1 5D25B026
-P 5900 3350
-F 0 "C700" H 6015 3396 50  0000 L CNN
-F 1 "220nF" H 6015 3305 50  0000 L CNN
-F 2 "Capacitor_SMD:C_0402_1005Metric" H 5938 3200 50  0001 C CNN
-F 3 "~" H 5900 3350 50  0001 C CNN
-	1    5900 3350
-	1    0    0    -1
-$EndComp
-$Comp
-L power:GND #PWR0277
-U 1 1 5D25C8C0
-P 5900 3500
-F 0 "#PWR0277" H 5900 3250 50  0001 C CNN
-F 1 "GND" H 5905 3327 50  0000 C CNN
-F 2 "" H 5900 3500 50  0001 C CNN
-F 3 "" H 5900 3500 50  0001 C CNN
-	1    5900 3500
-	1    0    0    -1
-$EndComp
-$Comp
-L power:+1V8 #PWR0278
-U 1 1 5D25D69D
-P 5900 3200
-F 0 "#PWR0278" H 5900 3050 50  0001 C CNN
-F 1 "+1V8" H 5915 3373 50  0000 C CNN
-F 2 "" H 5900 3200 50  0001 C CNN
-F 3 "" H 5900 3200 50  0001 C CNN
-	1    5900 3200
-	1    0    0    -1
-$EndComp
-Wire Wire Line
-	5900 3200 6000 3200
-Connection ~ 5900 3200
-Wire Wire Line
-	6300 3200 6400 3200
-Connection ~ 6400 3200
-Wire Wire Line
-	6400 3200 6800 3200
 Connection ~ 6800 3200
 Wire Wire Line
@@
 Wire Wire Line
 	7200 3500 6800 3500
-Connection ~ 5900 3500
-Connection ~ 6400 3500
-Wire Wire Line
-	6400 3500 5900 3500
 Connection ~ 6800 3500
-Wire Wire Line
-	6800 3500 6400 3500
 Wire Wire Line
 	7600 3200 7600 3700
@@
 L Switch:SW_Push SW702
 U 1 1 5D27E22C
-P 4500 6200
-F 0 "SW702" H 4500 6485 50  0000 C CNN
-F 1 "SW_Push" H 4500 6394 50  0000 C CNN
-F 2 "footprints:contact" H 4500 6400 50  0001 C CNN
-F 3 "~" H 4500 6400 50  0001 C CNN
-	1    4500 6200
+P 5000 6200
+F 0 "SW702" H 5000 6485 50  0000 C CNN
+F 1 "SW_Push" H 5000 6394 50  0000 C CNN
+F 2 "footprints:contact" H 5000 6400 50  0001 C CNN
+F 3 "~" H 5000 6400 50  0001 C CNN
+	1    5000 6200
 	1    0    0    -1
 $EndComp
@@
 L Switch:SW_Push SW703
 U 1 1 5D27EABD
-P 5000 6600
-F 0 "SW703" H 5000 6885 50  0000 C CNN
-F 1 "SW_Push" H 5000 6794 50  0000 C CNN
-F 2 "footprints:contact" H 5000 6800 50  0001 C CNN
-F 3 "~" H 5000 6800 50  0001 C CNN
-	1    5000 6600
+P 4600 6600
+F 0 "SW703" H 4600 6885 50  0000 C CNN
+F 1 "SW_Push" H 4600 6794 50  0000 C CNN
+F 2 "footprints:contact" H 4600 6800 50  0001 C CNN
+F 3 "~" H 4600 6800 50  0001 C CNN
+	1    4600 6600
 	1    0    0    -1
 $EndComp
@@
 	1    0    0    -1
 $EndComp
-Text Label 2900 5500 0    50   ~ 0
-SW_SE
-Text Label 3700 5500 0    50   ~ 0
-SW_ST
-Text Label 2700 6000 0    50   ~ 0
-SW_UP
-Text Label 2200 6400 0    50   ~ 0
-SW_LE
-Text Label 3200 6400 0    50   ~ 0
-SW_RI
-Text Label 2700 6800 0    50   ~ 0
-SW_DN
-Text Label 4100 6200 0    50   ~ 0
-SW_A
-Text Label 4600 6600 0    50   ~ 0
-SW_B
 $Comp
 L power:GND #PWR0281
@@
 L power:GND #PWR0283
 U 1 1 5D28AA10
-P 4700 6200
-F 0 "#PWR0283" H 4700 5950 50  0001 C CNN
-F 1 "GND" H 4705 6027 50  0000 C CNN
-F 2 "" H 4700 6200 50  0001 C CNN
-F 3 "" H 4700 6200 50  0001 C CNN
-	1    4700 6200
+P 5200 6200
+F 0 "#PWR0283" H 5200 5950 50  0001 C CNN
+F 1 "GND" H 5205 6027 50  0000 C CNN
+F 2 "" H 5200 6200 50  0001 C CNN
+F 3 "" H 5200 6200 50  0001 C CNN
+	1    5200 6200
 	1    0    0    -1
 $EndComp
@@
 L power:GND #PWR0284
 U 1 1 5D28AD69
-P 5200 6600
-F 0 "#PWR0284" H 5200 6350 50  0001 C CNN
-F 1 "GND" H 5205 6427 50  0000 C CNN
-F 2 "" H 5200 6600 50  0001 C CNN
-F 3 "" H 5200 6600 50  0001 C CNN
-	1    5200 6600
+P 4800 6600
+F 0 "#PWR0284" H 4800 6350 50  0001 C CNN
+F 1 "GND" H 4805 6427 50  0000 C CNN
+F 2 "" H 4800 6600 50  0001 C CNN
+F 3 "" H 4800 6600 50  0001 C CNN
+	1    4800 6600
 	1    0    0    -1
 $EndComp
@@
 	1    0    0    -1
 $EndComp
-Wire Wire Line
-	2700 6000 2900 6000
-Wire Wire Line
-	2900 5500 3100 5500
-Wire Wire Line
-	2200 6400 2400 6400
-Wire Wire Line
-	2700 6800 2900 6800
-Wire Wire Line
-	3200 6400 3400 6400
-Wire Wire Line
-	4100 6200 4300 6200
-Wire Wire Line
-	3700 5500 3900 5500
-Wire Wire Line
-	4600 6600 4800 6600
-Text Label 4000 3000 0    50   ~ 0
-SW_SE
-Wire Wire Line
-	4000 3000 4200 3000
-Text Label 4000 3100 0    50   ~ 0
-SW_ST
-Wire Wire Line
-	4000 3100 4200 3100
-Text Label 4000 3200 0    50   ~ 0
-SW_A
-Wire Wire Line
-	4000 3200 4200 3200
-Text Label 4000 3300 0    50   ~ 0
-SW_B
-Wire Wire Line
-	4000 3300 4200 3300
-Text Label 4000 3400 0    50   ~ 0
-SW_UP
-Wire Wire Line
-	4000 3400 4200 3400
-Text Label 4000 3500 0    50   ~ 0
-SW_LE
-Wire Wire Line
-	4000 3500 4200 3500
-Text Label 4000 3600 0    50   ~ 0
-SW_RI
-Wire Wire Line
-	4000 3600 4200 3600
-Text Label 4000 3700 0    50   ~ 0
-SW_DN
-Wire Wire Line
-	4000 3700 4200 3700
 NoConn ~ 9300 3400
 NoConn ~ 9300 3500
+$Comp
+L Device:L L700
+U 1 1 5D259B1C
+P 6550 3200
+F 0 "L700" V 6740 3200 50  0000 C CNN
+F 1 "120R" V 6649 3200 50  0000 C CNN
+F 2 "Inductor_SMD:L_0603_1608Metric" H 6550 3200 50  0001 C CNN
+F 3 "~" H 6550 3200 50  0001 C CNN
+	1    6550 3200
+	0    -1   -1   0
+$EndComp
+$Comp
+L Device:C C700
+U 1 1 5D25B026
+P 6300 3350
+F 0 "C700" H 6415 3396 50  0000 L CNN
+F 1 "220nF" H 6415 3305 50  0000 L CNN
+F 2 "Capacitor_SMD:C_0402_1005Metric" H 6338 3200 50  0001 C CNN
+F 3 "~" H 6300 3350 50  0001 C CNN
+	1    6300 3350
+	1    0    0    -1
+$EndComp
+$Comp
+L power:GND #PWR0277
+U 1 1 5D25C8C0
+P 6300 3500
+F 0 "#PWR0277" H 6300 3250 50  0001 C CNN
+F 1 "GND" H 6305 3327 50  0000 C CNN
+F 2 "" H 6300 3500 50  0001 C CNN
+F 3 "" H 6300 3500 50  0001 C CNN
+	1    6300 3500
+	1    0    0    -1
+$EndComp
+$Comp
+L power:+1V8 #PWR0278
+U 1 1 5D25D69D
+P 6300 3200
+F 0 "#PWR0278" H 6300 3050 50  0001 C CNN
+F 1 "+1V8" H 6315 3373 50  0000 C CNN
+F 2 "" H 6300 3200 50  0001 C CNN
+F 3 "" H 6300 3200 50  0001 C CNN
+	1    6300 3200
+	1    0    0    -1
+$EndComp
+Wire Wire Line
+	6300 3200 6400 3200
+Connection ~ 6300 3200
+Connection ~ 6300 3500
+Wire Wire Line
+	6700 3200 6800 3200
+Wire Wire Line
+	6300 3500 6800 3500
+Text GLabel 2900 6800 0    50   Output ~ 0
+SW_DN
+Text GLabel 3100 5500 0    50   Output ~ 0
+SW_SE
+Text GLabel 2900 6000 0    50   Output ~ 0
+SW_UP
+Text GLabel 2400 6400 0    50   Output ~ 0
+SW_LE
+Text GLabel 4400 6600 0    50   Output ~ 0
+SW_B
+Text GLabel 4800 6200 0    50   Output ~ 0
+SW_A
+Text GLabel 3400 6400 0    50   Output ~ 0
+SW_RI
+Text GLabel 3900 5500 0    50   Output ~ 0
+SW_ST
 $EndSCHEMATC

Commit message: pcb: routing
Parts:
- C700, C702, C703: symbol Device:C -> pcb-rescue:C-Device
- L700: symbol Device:L -> pcb-rescue:L-Device
- R700: symbol Device:R -> pcb-rescue:R-Device
- SW700, SW701, SW702, SW703, SW704, SW705, SW706, SW707: symbol Switch:SW_Push -> pcb-rescue:SW_Push-Switch
Changed lines of the file:
@@
 	4000 4600 4200 4600
 $Comp
-L Device:C C703
+L pcb-rescue:C-Device C703
 U 1 1 5D254E8F
 P 7200 3350
@@
 $EndComp
 $Comp
-L Device:C C702
+L pcb-rescue:C-Device C702
 U 1 1 5D256675
 P 6800 3350
@@
 	9300 3300 9500 3300
 $Comp
-L Device:R R700
+L pcb-rescue:R-Device R700
 U 1 1 5D26F11D
 P 9400 4650
@@
 $EndComp
 $Comp
-L power:GND #PWR0279
+L pcb-rescue:GND-power #PWR0279
 U 1 1 5D270686
 P 9400 4800
@@
 	9400 4400 9400 4500
 $Comp
-L power:GND #PWR0280
+L pcb-rescue:GND-power #PWR0280
 U 1 1 5D271CAD
 P 9400 4100
@@
 	9400 3800 9400 3900
 $Comp
-L Switch:SW_Push SW704
+L pcb-rescue:SW_Push-Switch SW704
 U 1 1 5D2797BD
 P 3100 6000
@@
 $EndComp
 $Comp
-L Switch:SW_Push SW705
+L pcb-rescue:SW_Push-Switch SW705
 U 1 1 5D27BD89
 P 2600 6400
@@
 $EndComp
 $Comp
-L Switch:SW_Push SW707
+L pcb-rescue:SW_Push-Switch SW707
 U 1 1 5D27CCB2
 P 3100 6800
@@
 $EndComp
 $Comp
-L Switch:SW_Push SW706
+L pcb-rescue:SW_Push-Switch SW706
 U 1 1 5D27D8DE
 P 3600 6400
@@
 $EndComp
 $Comp
-L Switch:SW_Push SW702
+L pcb-rescue:SW_Push-Switch SW702
 U 1 1 5D27E22C
 P 5000 6200
@@
 $EndComp
 $Comp
-L Switch:SW_Push SW703
+L pcb-rescue:SW_Push-Switch SW703
 U 1 1 5D27EABD
 P 4600 6600
@@
 $EndComp
 $Comp
-L Switch:SW_Push SW700
+L pcb-rescue:SW_Push-Switch SW700
 U 1 1 5D281FA3
 P 3300 5500
@@
 $EndComp
 $Comp
-L Switch:SW_Push SW701
+L pcb-rescue:SW_Push-Switch SW701
 U 1 1 5D2828BB
 P 4100 5500
@@
 $EndComp
 $Comp
-L power:GND #PWR0281
+L pcb-rescue:GND-power #PWR0281
 U 1 1 5D288EE2
 P 4300 5500
@@
 $EndComp
 $Comp
-L power:GND #PWR0282
+L pcb-rescue:GND-power #PWR0282
 U 1 1 5D289F76
 P 3500 5500
@@
 $EndComp
 $Comp
-L power:GND #PWR0283
+L pcb-rescue:GND-power #PWR0283
 U 1 1 5D28AA10
 P 5200 6200
@@
 $EndComp
 $Comp
-L power:GND #PWR0284
+L pcb-rescue:GND-power #PWR0284
 U 1 1 5D28AD69
 P 4800 6600
@@
 $EndComp
 $Comp
-L power:GND #PWR0285
+L pcb-rescue:GND-power #PWR0285
 U 1 1 5D28B128
 P 3800 6400
@@
 $EndComp
 $Comp
-L power:GND #PWR0286
+L pcb-rescue:GND-power #PWR0286
 U 1 1 5D28B509
 P 3300 6800
@@
 $EndComp
 $Comp
-L power:GND #PWR0287
+L pcb-rescue:GND-power #PWR0287
 U 1 1 5D28B91D
 P 2800 6400
@@
 $EndComp
 $Comp
-L power:GND #PWR0288
+L pcb-rescue:GND-power #PWR0288
 U 1 1 5D28BC76
 P 3300 6000
@@
 NoConn ~ 9300 3500
 $Comp
-L Device:L L700
+L pcb-rescue:L-Device L700
 U 1 1 5D259B1C
 P 6550 3200
@@
 $EndComp
 $Comp
-L Device:C C700
+L pcb-rescue:C-Device C700
 U 1 1 5D25B026
 P 6300 3350
@@
 $EndComp
 $Comp
-L power:GND #PWR0277
+L pcb-rescue:GND-power #PWR0277
 U 1 1 5D25C8C0
 P 6300 3500
@@
 $EndComp
 $Comp
-L power:+1V8 #PWR0278
+L pcb-rescue:+1V8-power #PWR0278
 U 1 1 5D25D69D
 P 6300 3200

Commit message: pcb: rev 0.1
Parts:
- C700, C702, C703: symbol pcb-rescue:C-Device -> pcb-rescue:C-Device-pcb-rescue
- L700: symbol pcb-rescue:L-Device -> pcb-rescue:L-Device-pcb-rescue
- R700: symbol pcb-rescue:R-Device -> pcb-rescue:R-Device-pcb-rescue
- SW700, SW701, SW702, SW703, SW704, SW705, SW706, SW707: symbol pcb-rescue:SW_Push-Switch -> pcb-rescue:SW_Push-Switch-pcb-rescue
Changed lines of the file:
@@
 encoding utf-8
 Sheet 8 11
-Title "Keypad & GPIO"
-Date ""
+Title "RhythmPocket"
+Date "2019-07-16"
 Rev "R0.1"
 Comp "ZephRay"
@@
 	4000 4600 4200 4600
 $Comp
-L pcb-rescue:C-Device C703
+L pcb-rescue:C-Device-pcb-rescue C703
 U 1 1 5D254E8F
 P 7200 3350
@@
 $EndComp
 $Comp
-L pcb-rescue:C-Device C702
+L pcb-rescue:C-Device-pcb-rescue C702
 U 1 1 5D256675
 P 6800 3350
@@
 	9300 3300 9500 3300
 $Comp
-L pcb-rescue:R-Device R700
+L pcb-rescue:R-Device-pcb-rescue R700
 U 1 1 5D26F11D
 P 9400 4650
@@
 $EndComp
 $Comp
-L pcb-rescue:GND-power #PWR0279
+L pcb-rescue:GND-power-pcb-rescue #PWR0279
 U 1 1 5D270686
 P 9400 4800
@@
 	9400 4400 9400 4500
 $Comp
-L pcb-rescue:GND-power #PWR0280
+L pcb-rescue:GND-power-pcb-rescue #PWR0280
 U 1 1 5D271CAD
 P 9400 4100
@@
 	9400 3800 9400 3900
 $Comp
-L pcb-rescue:SW_Push-Switch SW704
+L pcb-rescue:SW_Push-Switch-pcb-rescue SW704
 U 1 1 5D2797BD
 P 3100 6000
@@
 $EndComp
 $Comp
-L pcb-rescue:SW_Push-Switch SW705
+L pcb-rescue:SW_Push-Switch-pcb-rescue SW705
 U 1 1 5D27BD89
 P 2600 6400
@@
 $EndComp
 $Comp
-L pcb-rescue:SW_Push-Switch SW707
+L pcb-rescue:SW_Push-Switch-pcb-rescue SW707
 U 1 1 5D27CCB2
 P 3100 6800
@@
 $EndComp
 $Comp
-L pcb-rescue:SW_Push-Switch SW706
+L pcb-rescue:SW_Push-Switch-pcb-rescue SW706
 U 1 1 5D27D8DE
 P 3600 6400
@@
 $EndComp
 $Comp
-L pcb-rescue:SW_Push-Switch SW702
+L pcb-rescue:SW_Push-Switch-pcb-rescue SW702
 U 1 1 5D27E22C
 P 5000 6200
@@
 $EndComp
 $Comp
-L pcb-rescue:SW_Push-Switch SW703
+L pcb-rescue:SW_Push-Switch-pcb-rescue SW703
 U 1 1 5D27EABD
 P 4600 6600
@@
 $EndComp
 $Comp
-L pcb-rescue:SW_Push-Switch SW700
+L pcb-rescue:SW_Push-Switch-pcb-rescue SW700
 U 1 1 5D281FA3
 P 3300 5500
@@
 $EndComp
 $Comp
-L pcb-rescue:SW_Push-Switch SW701
+L pcb-rescue:SW_Push-Switch-pcb-rescue SW701
 U 1 1 5D2828BB
 P 4100 5500
@@
 $EndComp
 $Comp
-L pcb-rescue:GND-power #PWR0281
+L pcb-rescue:GND-power-pcb-rescue #PWR0281
 U 1 1 5D288EE2
 P 4300 5500
@@
 $EndComp
 $Comp
-L pcb-rescue:GND-power #PWR0282
+L pcb-rescue:GND-power-pcb-rescue #PWR0282
 U 1 1 5D289F76
 P 3500 5500
@@
 $EndComp
 $Comp
-L pcb-rescue:GND-power #PWR0283
+L pcb-rescue:GND-power-pcb-rescue #PWR0283
 U 1 1 5D28AA10
 P 5200 6200
@@
 $EndComp
 $Comp
-L pcb-rescue:GND-power #PWR0284
+L pcb-rescue:GND-power-pcb-rescue #PWR0284
 U 1 1 5D28AD69
 P 4800 6600
@@
 $EndComp
 $Comp
-L pcb-rescue:GND-power #PWR0285
+L pcb-rescue:GND-power-pcb-rescue #PWR0285
 U 1 1 5D28B128
 P 3800 6400
@@
 $EndComp
 $Comp
-L pcb-rescue:GND-power #PWR0286
+L pcb-rescue:GND-power-pcb-rescue #PWR0286
 U 1 1 5D28B509
 P 3300 6800
@@
 $EndComp
 $Comp
-L pcb-rescue:GND-power #PWR0287
+L pcb-rescue:GND-power-pcb-rescue #PWR0287
 U 1 1 5D28B91D
 P 2800 6400
@@
 $EndComp
 $Comp
-L pcb-rescue:GND-power #PWR0288
+L pcb-rescue:GND-power-pcb-rescue #PWR0288
 U 1 1 5D28BC76
 P 3300 6000
@@
 NoConn ~ 9300 3500
 $Comp
-L pcb-rescue:L-Device L700
+L pcb-rescue:L-Device-pcb-rescue L700
 U 1 1 5D259B1C
 P 6550 3200
@@
 $EndComp
 $Comp
-L pcb-rescue:C-Device C700
+L pcb-rescue:C-Device-pcb-rescue C700
 U 1 1 5D25B026
 P 6300 3350
@@
 $EndComp
 $Comp
-L pcb-rescue:GND-power #PWR0277
+L pcb-rescue:GND-power-pcb-rescue #PWR0277
 U 1 1 5D25C8C0
 P 6300 3500
@@
 $EndComp
 $Comp
-L pcb-rescue:+1V8-power #PWR0278
+L pcb-rescue:+1V8-power-pcb-rescue #PWR0278
 U 1 1 5D25D69D
 P 6300 3200
