File: pcb/keypad.sch (KiCad schematic (older format))
At the start: 14 parts, among them SW700 SW_Push, SW701 SW_Push, SW702 SW_Push, SW703 SW_Push, SW704 SW_Push, SW705 SW_Push, SW706 SW_Push, SW707 SW_Push, U100 MCIMX7S5EVM08SC

Commit message: pcb: remap schematic symbols
Parts:
- C700, C702, C703: symbol pcb-rescue:C-Device-pcb-rescue -> Device:C
- L700: symbol pcb-rescue:L-Device-pcb-rescue -> Device:L_Small
- R700: symbol pcb-rescue:R-Device-pcb-rescue -> Device:R
- SW700, SW701, SW702, SW703, SW704, SW705, SW706, SW707: symbol pcb-rescue:SW_Push-Switch-pcb-rescue -> Switch:SW_Push
Changed lines of the file:
@@
 	4000 4600 4200 4600
 $Comp
-L pcb-rescue:C-Device-pcb-rescue C703
+L Device:C C703
 U 1 1 5D254E8F
 P 7200 3350
@@
 $EndComp
 $Comp
-L pcb-rescue:C-Device-pcb-rescue C702
+L Device:C C702
 U 1 1 5D256675
 P 6800 3350
@@
 	9300 3300 9500 3300
 $Comp
-L pcb-rescue:R-Device-pcb-rescue R700
+L Device:R R700
 U 1 1 5D26F11D
 P 9400 4650
@@
 $EndComp
 $Comp
-L pcb-rescue:GND-power-pcb-rescue #PWR0279
+L power:GND #PWR0279
 U 1 1 5D270686
 P 9400 4800
@@
 	9400 4400 9400 4500
 $Comp
-L pcb-rescue:GND-power-pcb-rescue #PWR0280
+L power:GND #PWR0280
 U 1 1 5D271CAD
 P 9400 4100
@@
 	9400 3800 9400 3900
 $Comp
-L pcb-rescue:SW_Push-Switch-pcb-rescue SW704
+L Switch:SW_Push SW704
 U 1 1 5D2797BD
 P 3100 6000
@@
 $EndComp
 $Comp
-L pcb-rescue:SW_Push-Switch-pcb-rescue SW705
+L Switch:SW_Push SW705
 U 1 1 5D27BD89
 P 2600 6400
@@
 $EndComp
 $Comp
-L pcb-rescue:SW_Push-Switch-pcb-rescue SW707
+L Switch:SW_Push SW707
 U 1 1 5D27CCB2
 P 3100 6800
@@
 $EndComp
 $Comp
-L pcb-rescue:SW_Push-Switch-pcb-rescue SW706
+L Switch:SW_Push SW706
 U 1 1 5D27D8DE
 P 3600 6400
@@
 $EndComp
 $Comp
-L pcb-rescue:SW_Push-Switch-pcb-rescue SW702
+L Switch:SW_Push SW702
 U 1 1 5D27E22C
 P 5000 6200
@@
 $EndComp
 $Comp
-L pcb-rescue:SW_Push-Switch-pcb-rescue SW703
+L Switch:SW_Push SW703
 U 1 1 5D27EABD
 P 4600 6600
@@
 $EndComp
 $Comp
-L pcb-rescue:SW_Push-Switch-pcb-rescue SW700
+L Switch:SW_Push SW700
 U 1 1 5D281FA3
 P 3300 5500
@@
 $EndComp
 $Comp
-L pcb-rescue:SW_Push-Switch-pcb-rescue SW701
+L Switch:SW_Push SW701
 U 1 1 5D2828BB
 P 4100 5500
@@
 $EndComp
 $Comp
-L pcb-rescue:GND-power-pcb-rescue #PWR0281
+L power:GND #PWR0281
 U 1 1 5D288EE2
 P 4300 5500
@@
 $EndComp
 $Comp
-L pcb-rescue:GND-power-pcb-rescue #PWR0282
+L power:GND #PWR0282
 U 1 1 5D289F76
 P 3500 5500
@@
 $EndComp
 $Comp
-L pcb-rescue:GND-power-pcb-rescue #PWR0283
+L power:GND #PWR0283
 U 1 1 5D28AA10
 P 5200 6200
@@
 $EndComp
 $Comp
-L pcb-rescue:GND-power-pcb-rescue #PWR0284
+L power:GND #PWR0284
 U 1 1 5D28AD69
 P 4800 6600
@@
 $EndComp
 $Comp
-L pcb-rescue:GND-power-pcb-rescue #PWR0285
+L power:GND #PWR0285
 U 1 1 5D28B128
 P 3800 6400
@@
 $EndComp
 $Comp
-L pcb-rescue:GND-power-pcb-rescue #PWR0286
+L power:GND #PWR0286
 U 1 1 5D28B509
 P 3300 6800
@@
 $EndComp
 $Comp
-L pcb-rescue:GND-power-pcb-rescue #PWR0287
+L power:GND #PWR0287
 U 1 1 5D28B91D
 P 2800 6400
@@
 $EndComp
 $Comp
-L pcb-rescue:GND-power-pcb-rescue #PWR0288
+L power:GND #PWR0288
 U 1 1 5D28BC76
 P 3300 6000
@@
 NoConn ~ 9300 3500
 $Comp
-L pcb-rescue:L-Device-pcb-rescue L700
+L Device:L_Small L700
 U 1 1 5D259B1C
 P 6550 3200
@@
 $EndComp
 $Comp
-L pcb-rescue:C-Device-pcb-rescue C700
+L Device:C C700
 U 1 1 5D25B026
 P 6300 3350
@@
 $EndComp
 $Comp
-L pcb-rescue:GND-power-pcb-rescue #PWR0277
+L power:GND #PWR0277
 U 1 1 5D25C8C0
 P 6300 3500
@@
 $EndComp
 $Comp
-L pcb-rescue:+1V8-power-pcb-rescue #PWR0278
+L power:+1V8 #PWR0278
 U 1 1 5D25D69D
 P 6300 3200

Commit message: pcb: bug fixes
Parts:
- L700: symbol Device:L_Small -> Device:L
Changed lines of the file:
@@
 NoConn ~ 9300 3500
 $Comp
-L Device:L_Small L700
+L Device:L L700
 U 1 1 5D259B1C
 P 6550 3200
