File: pcb/lcd.sch (KiCad schematic (older format))
At the start: 37 parts, among them J500 FPC_18P_1.0MM, Q500 IRLML6402, U100 MCIMX7S5EVM08SC, U500 XC2C32A_QF32, U501 ADP5075, U502 LM324

Commit message: pcb: rev 0.1
Parts:
- C500, C501, C502, C503, C504, C505, C506, C507, C508, C509, C510, C511, C512: symbol pcb-rescue:C-Device -> pcb-rescue:C-Device-pcb-rescue
- D500, D501: symbol pcb-rescue:D_Schottky-Device -> pcb-rescue:D_Schottky-Device-pcb-rescue
- J500: symbol pcb-rescue:Conn_01x18-Connector_Generic -> pcb-rescue:Conn_01x18-Connector_Generic-pcb-rescue
- L500: symbol pcb-rescue:L-Device -> pcb-rescue:L-Device-pcb-rescue
- Q500: symbol pcb-rescue:IRLML6402-Transistor_FET -> pcb-rescue:IRLML6402-Transistor_FET-pcb-rescue
- R500, R501, R502, R503, R504, R505, R506, R507, R508, R509: symbol pcb-rescue:R-Device -> pcb-rescue:R-Device-pcb-rescue
- RN500, RN501, RN502, RN503: symbol pcb-rescue:R_Pack04-Device -> pcb-rescue:R_Pack04-Device-pcb-rescue
- RV500: symbol pcb-rescue:R_POT-Device -> pcb-rescue:R_POT-Device-pcb-rescue
- U502: symbol pcb-rescue:LM324-Amplifier_Operational -> pcb-rescue:LM324-Amplifier_Operational-pcb-rescue
Changed lines of the file:
@@
 encoding utf-8
 Sheet 6 11
-Title "STN LCD"
-Date ""
+Title "RhythmPocket"
+Date "2019-07-16"
 Rev "R0.1"
 Comp "ZephRay"
@@
 	3600 2000 3700 2000
 $Comp
-L pcb-rescue:R_Pack04-Device RN500
+L pcb-rescue:R_Pack04-Device-pcb-rescue RN500
 U 1 1 5D423DF0
 P 5200 1600
@@
 $EndComp
 $Comp
-L pcb-rescue:R_Pack04-Device RN501
+L pcb-rescue:R_Pack04-Device-pcb-rescue RN501
 U 1 1 5D4288BB
 P 5200 2000
@@
 $EndComp
 $Comp
-L pcb-rescue:R_Pack04-Device RN503
+L pcb-rescue:R_Pack04-Device-pcb-rescue RN503
 U 1 1 5D42C7E0
 P 7100 2000
@@
 	7200 2800 6800 2800
 $Comp
-L pcb-rescue:GND-power #PWR0223
+L pcb-rescue:GND-power-pcb-rescue #PWR0223
 U 1 1 5D454409
 P 6900 3300
@@
 	6900 3100 6900 3200
 $Comp
-L pcb-rescue:C-Device C?
+L pcb-rescue:C-Device-pcb-rescue C?
 U 1 1 5D47BA54
 P 1400 1050
@@
 $EndComp
 $Comp
-L pcb-rescue:GND-power #PWR?
+L pcb-rescue:GND-power-pcb-rescue #PWR?
 U 1 1 5D47BA5A
 P 1400 1300
@@
 	1400 1300 1400 1200
 $Comp
-L pcb-rescue:+1V8-power #PWR0231
+L pcb-rescue:+1V8-power-pcb-rescue #PWR0231
 U 1 1 5D47EFB1
 P 1400 700
@@
 Connection ~ 1400 700
 $Comp
-L pcb-rescue:C-Device C?
+L pcb-rescue:C-Device-pcb-rescue C?
 U 1 1 5D4808D9
 P 1400 4250
@@
 $EndComp
 $Comp
-L pcb-rescue:GND-power #PWR?
+L pcb-rescue:GND-power-pcb-rescue #PWR?
 U 1 1 5D4808DF
 P 1400 4500
@@
 	1400 4500 1400 4400
 $Comp
-L pcb-rescue:+1V8-power #PWR0233
+L pcb-rescue:+1V8-power-pcb-rescue #PWR0233
 U 1 1 5D4808E8
 P 1400 3900
@@
 Connection ~ 1400 3900
 $Comp
-L pcb-rescue:C-Device C?
+L pcb-rescue:C-Device-pcb-rescue C?
 U 1 1 5D483C06
 P 1400 5950
@@
 $EndComp
 $Comp
-L pcb-rescue:GND-power #PWR?
+L pcb-rescue:GND-power-pcb-rescue #PWR?
 U 1 1 5D483C0C
 P 1400 6200
@@
 	1400 6200 1400 6100
 $Comp
-L pcb-rescue:+1V8-power #PWR0235
+L pcb-rescue:+1V8-power-pcb-rescue #PWR0235
 U 1 1 5D483C15
 P 1400 5600
@@
 Connection ~ 1400 5600
 $Comp
-L pcb-rescue:C-Device C?
+L pcb-rescue:C-Device-pcb-rescue C?
 U 1 1 5D489120
 P 1400 7450
@@
 $EndComp
 $Comp
-L pcb-rescue:GND-power #PWR?
+L pcb-rescue:GND-power-pcb-rescue #PWR?
 U 1 1 5D489128
 P 1400 7600
@@
 $EndComp
 $Comp
-L pcb-rescue:Conn_01x18-Connector_Generic J500
+L pcb-rescue:Conn_01x18-Connector_Generic-pcb-rescue J500
 U 1 1 5D4BB38B
 P 9600 1600
@@
 $EndComp
 $Comp
-L pcb-rescue:GND-power #PWR0237
+L pcb-rescue:GND-power-pcb-rescue #PWR0237
 U 1 1 5D4BF290
 P 9300 2500
@@
 Connection ~ 4500 6100
 $Comp
-L pcb-rescue:C-Device C508
+L pcb-rescue:C-Device-pcb-rescue C508
 U 1 1 5D5F56B0
 P 4250 6100
@@
 $EndComp
 $Comp
-L pcb-rescue:GND-power #PWR0238
+L pcb-rescue:GND-power-pcb-rescue #PWR0238
 U 1 1 5D5FB1D3
 P 4000 6100
@@
 	4000 6100 4100 6100
 $Comp
-L pcb-rescue:+3V3-power #PWR?
+L pcb-rescue:+3V3-power-pcb-rescue #PWR?
 U 1 1 5D622DCE
 P 5400 4600
@@
 $EndComp
 $Comp
-L pcb-rescue:IRLML6402-Transistor_FET Q?
+L pcb-rescue:IRLML6402-Transistor_FET-pcb-rescue Q?
 U 1 1 5D622DD4
 P 5300 4900
@@
 	5400 4600 5400 4700
 $Comp
-L pcb-rescue:R-Device R?
+L pcb-rescue:R-Device-pcb-rescue R?
 U 1 1 5D622DDB
 P 4900 5150
@@
 $EndComp
 $Comp
-L pcb-rescue:R-Device R?
+L pcb-rescue:R-Device-pcb-rescue R?
 U 1 1 5D622DE1
 P 4900 4650
@@
 	4900 5000 4900 4900
 $Comp
-L pcb-rescue:GND-power #PWR?
+L pcb-rescue:GND-power-pcb-rescue #PWR?
 U 1 1 5D622DED
 P 4900 5300
@@
 $EndComp
 $Comp
-L pcb-rescue:+3V3-power #PWR?
+L pcb-rescue:+3V3-power-pcb-rescue #PWR?
 U 1 1 5D622DF3
 P 4900 4500
@@
 $EndComp
 $Comp
-L pcb-rescue:D_Schottky-Device D?
+L pcb-rescue:D_Schottky-Device-pcb-rescue D?
 U 1 1 5D622DF9
 P 4650 4900
@@
 NoConn ~ 4600 6500
 $Comp
-L pcb-rescue:R-Device R502
+L pcb-rescue:R-Device-pcb-rescue R502
 U 1 1 5D672E77
 P 4350 6700
@@
 $EndComp
 $Comp
-L pcb-rescue:C-Device C509
+L pcb-rescue:C-Device-pcb-rescue C509
 U 1 1 5D673908
 P 3950 6700
@@
 $EndComp
 $Comp
-L pcb-rescue:C-Device C510
+L pcb-rescue:C-Device-pcb-rescue C510
 U 1 1 5D674718
 P 4300 7050
@@
 $EndComp
 $Comp
-L pcb-rescue:C-Device C511
+L pcb-rescue:C-Device-pcb-rescue C511
 U 1 1 5D6756DB
 P 6150 5600
@@
 $EndComp
 $Comp
-L pcb-rescue:R-Device R503
+L pcb-rescue:R-Device-pcb-rescue R503
 U 1 1 5D675D3D
 P 5800 6250
@@
 $EndComp
 $Comp
-L pcb-rescue:R-Device R509
+L pcb-rescue:R-Device-pcb-rescue R509
 U 1 1 5D67C719
 P 6150 6400
@@
 $EndComp
 $Comp
-L pcb-rescue:C-Device C512
+L pcb-rescue:C-Device-pcb-rescue C512
 U 1 1 5D67D52C
 P 6400 6850
@@
 $EndComp
 $Comp
-L pcb-rescue:D_Schottky-Device D501
+L pcb-rescue:D_Schottky-Device-pcb-rescue D501
 U 1 1 5D685CDF
 P 6150 6600
@@
 	6000 6600 5800 6600
 $Comp
-L pcb-rescue:GND-power #PWR?
+L pcb-rescue:GND-power-pcb-rescue #PWR?
 U 1 1 5D6AFE75
 P 6400 5600
@@
 	6300 5600 6400 5600
 $Comp
-L pcb-rescue:GND-power #PWR?
+L pcb-rescue:GND-power-pcb-rescue #PWR?
 U 1 1 5D6B732F
 P 6400 7000
@@
 $EndComp
 $Comp
-L pcb-rescue:GND-power #PWR?
+L pcb-rescue:GND-power-pcb-rescue #PWR?
 U 1 1 5D6B76FB
 P 5600 7200
@@
 $EndComp
 $Comp
-L pcb-rescue:GND-power #PWR?
+L pcb-rescue:GND-power-pcb-rescue #PWR?
 U 1 1 5D6B7A0D
 P 4600 7200
@@
 $EndComp
 $Comp
-L pcb-rescue:GND-power #PWR?
+L pcb-rescue:GND-power-pcb-rescue #PWR?
 U 1 1 5D6B80FB
 P 3800 6700
@@
 $EndComp
 $Comp
-L pcb-rescue:GND-power #PWR?
+L pcb-rescue:GND-power-pcb-rescue #PWR?
 U 1 1 5D6B8450
 P 4300 7200
@@
 NoConn ~ 5600 6800
 $Comp
-L pcb-rescue:L-Device L500
+L pcb-rescue:L-Device-pcb-rescue L500
 U 1 1 5D6F546B
 P 5800 6850
@@
 $EndComp
 $Comp
-L pcb-rescue:GND-power #PWR?
+L pcb-rescue:GND-power-pcb-rescue #PWR?
 U 1 1 5D6F67EF
 P 5800 7100
@@
 Connection ~ 6400 6400
 $Comp
-L pcb-rescue:R_POT-Device RV500
+L pcb-rescue:R_POT-Device-pcb-rescue RV500
 U 1 1 5D72C05F
 P 5800 5800
@@
 	7200 6000 7200 6050
 $Comp
-L pcb-rescue:R-Device R504
+L pcb-rescue:R-Device-pcb-rescue R504
 U 1 1 5D585916
 P 7200 6250
@@
 	6700 5750 6700 6400
 $Comp
-L pcb-rescue:LM324-Amplifier_Operational U502
+L pcb-rescue:LM324-Amplifier_Operational-pcb-rescue U502
 U 5 1 5D80D00D
 P 6800 5450
@@
 	7800 5050 7800 5150
 $Comp
-L pcb-rescue:LM324-Amplifier_Operational U502
+L pcb-rescue:LM324-Amplifier_Operational-pcb-rescue U502
 U 4 1 5D78D689
 P 8100 6150
@@
 $EndComp
 $Comp
-L pcb-rescue:LM324-Amplifier_Operational U502
+L pcb-rescue:LM324-Amplifier_Operational-pcb-rescue U502
 U 3 1 5D78AB11
 P 8100 5750
@@
 $EndComp
 $Comp
-L pcb-rescue:LM324-Amplifier_Operational U502
+L pcb-rescue:LM324-Amplifier_Operational-pcb-rescue U502
 U 2 1 5D787DB9
 P 8100 5350
@@
 $EndComp
 $Comp
-L pcb-rescue:LM324-Amplifier_Operational U502
+L pcb-rescue:LM324-Amplifier_Operational-pcb-rescue U502
 U 1 1 5D783130
 P 8100 4950
@@
 	7200 5700 7200 5650
 $Comp
-L pcb-rescue:R-Device R508
+L pcb-rescue:R-Device-pcb-rescue R508
 U 1 1 5D7560C1
 P 7200 4650
@@
 $EndComp
 $Comp
-L pcb-rescue:R-Device R507
+L pcb-rescue:R-Device-pcb-rescue R507
 U 1 1 5D755DDC
 P 7200 5050
@@
 $EndComp
 $Comp
-L pcb-rescue:R-Device R505
+L pcb-rescue:R-Device-pcb-rescue R505
 U 1 1 5D753D04
 P 7200 5850
@@
 -11.6V to -17.8V
 $Comp
-L pcb-rescue:R-Device R506
+L pcb-rescue:R-Device-pcb-rescue R506
 U 1 1 5D75597D
 P 7200 5450
@@
 $EndComp
 $Comp
-L pcb-rescue:+1V8-power #PWR0224
+L pcb-rescue:+1V8-power-pcb-rescue #PWR0224
 U 1 1 5D45A159
 P 5400 2800
@@
 $EndComp
 $Comp
-L pcb-rescue:+3V3-power #PWR0225
+L pcb-rescue:+3V3-power-pcb-rescue #PWR0225
 U 1 1 5D45AD93
 P 4600 2800
@@
 	5400 3000 5400 2800
 $Comp
-L pcb-rescue:C-Device C500
+L pcb-rescue:C-Device-pcb-rescue C500
 U 1 1 5D4632AC
 P 5400 3450
@@
 $EndComp
 $Comp
-L pcb-rescue:C-Device C501
+L pcb-rescue:C-Device-pcb-rescue C501
 U 1 1 5D463E9F
 P 5000 3450
@@
 $EndComp
 $Comp
-L pcb-rescue:C-Device C502
+L pcb-rescue:C-Device-pcb-rescue C502
 U 1 1 5D46402C
 P 4600 3450
@@
 $EndComp
 $Comp
-L pcb-rescue:C-Device C503
+L pcb-rescue:C-Device-pcb-rescue C503
 U 1 1 5D464243
 P 4200 3450
@@
 $EndComp
 $Comp
-L pcb-rescue:GND-power #PWR0226
+L pcb-rescue:GND-power-pcb-rescue #PWR0226
 U 1 1 5D468CD4
 P 5400 3600
@@
 $EndComp
 $Comp
-L pcb-rescue:GND-power #PWR0227
+L pcb-rescue:GND-power-pcb-rescue #PWR0227
 U 1 1 5D46903A
 P 5000 3600
@@
 $EndComp
 $Comp
-L pcb-rescue:GND-power #PWR0228
+L pcb-rescue:GND-power-pcb-rescue #PWR0228
 U 1 1 5D46925D
 P 4600 3600
@@
 $EndComp
 $Comp
-L pcb-rescue:GND-power #PWR0229
+L pcb-rescue:GND-power-pcb-rescue #PWR0229
 U 1 1 5D4694F7
 P 4200 3600
@@
 	7300 2000 7700 2000
 $Comp
-L pcb-rescue:R_Pack04-Device RN502
+L pcb-rescue:R_Pack04-Device-pcb-rescue RN502
 U 1 1 5D42A1C4
 P 7100 1600
