File: pcb/lcd.sch (KiCad schematic (older format))
At the start: 37 parts, among them J500 FPC_18P_1.0MM, Q500 IRLML6402, U100 MCIMX7S5EVM08SC, U500 XC2C32A_QF32, U501 ADP5075, U502 LM324

Commit message: pcb: remap schematic symbols
Parts:
- C500, C501, C502, C503, C504, C505, C506, C507, C508, C509, C510, C511, C512: symbol pcb-rescue:C-Device-pcb-rescue -> Device:C
- D500, D501: symbol pcb-rescue:D_Schottky-Device-pcb-rescue -> Device:D_Schottky
- J500: symbol pcb-rescue:Conn_01x18-Connector_Generic-pcb-rescue -> Connector_Generic:Conn_01x18
- L500: symbol pcb-rescue:L-Device-pcb-rescue -> Device:L_Small
- Q500: symbol pcb-rescue:IRLML6402-Transistor_FET-pcb-rescue -> Transistor_FET:IRLML6402
- R500, R501, R502, R503, R504, R505, R506, R507, R508, R509: symbol pcb-rescue:R-Device-pcb-rescue -> Device:R
- RN500, RN501, RN502, RN503: symbol pcb-rescue:R_Pack04-Device-pcb-rescue -> Device:R_Pack04
- RV500: symbol pcb-rescue:R_POT-Device-pcb-rescue -> Device:R_POT
- U502: symbol pcb-rescue:LM324-Amplifier_Operational-pcb-rescue -> Amplifier_Operational:LM324
Changed lines of the file:
@@
 	3600 2000 3700 2000
 $Comp
-L pcb-rescue:R_Pack04-Device-pcb-rescue RN500
+L Device:R_Pack04 RN500
 U 1 1 5D423DF0
 P 5200 1600
@@
 $EndComp
 $Comp
-L pcb-rescue:R_Pack04-Device-pcb-rescue RN501
+L Device:R_Pack04 RN501
 U 1 1 5D4288BB
 P 5200 2000
@@
 $EndComp
 $Comp
-L pcb-rescue:R_Pack04-Device-pcb-rescue RN503
+L Device:R_Pack04 RN503
 U 1 1 5D42C7E0
 P 7100 2000
@@
 	7200 2800 6800 2800
 $Comp
-L pcb-rescue:GND-power-pcb-rescue #PWR0223
+L power:GND #PWR0223
 U 1 1 5D454409
 P 6900 3300
@@
 	6900 3100 6900 3200
 $Comp
-L pcb-rescue:C-Device-pcb-rescue C?
+L Device:C C?
 U 1 1 5D47BA54
 P 1400 1050
@@
 $EndComp
 $Comp
-L pcb-rescue:GND-power-pcb-rescue #PWR?
+L power:GND #PWR?
 U 1 1 5D47BA5A
 P 1400 1300
@@
 	1400 1300 1400 1200
 $Comp
-L pcb-rescue:+1V8-power-pcb-rescue #PWR0231
+L power:+1V8 #PWR0231
 U 1 1 5D47EFB1
 P 1400 700
@@
 Connection ~ 1400 700
 $Comp
-L pcb-rescue:C-Device-pcb-rescue C?
+L Device:C C?
 U 1 1 5D4808D9
 P 1400 4250
@@
 $EndComp
 $Comp
-L pcb-rescue:GND-power-pcb-rescue #PWR?
+L power:GND #PWR?
 U 1 1 5D4808DF
 P 1400 4500
@@
 	1400 4500 1400 4400
 $Comp
-L pcb-rescue:+1V8-power-pcb-rescue #PWR0233
+L power:+1V8 #PWR0233
 U 1 1 5D4808E8
 P 1400 3900
@@
 Connection ~ 1400 3900
 $Comp
-L pcb-rescue:C-Device-pcb-rescue C?
+L Device:C C?
 U 1 1 5D483C06
 P 1400 5950
@@
 $EndComp
 $Comp
-L pcb-rescue:GND-power-pcb-rescue #PWR?
+L power:GND #PWR?
 U 1 1 5D483C0C
 P 1400 6200
@@
 	1400 6200 1400 6100
 $Comp
-L pcb-rescue:+1V8-power-pcb-rescue #PWR0235
+L power:+1V8 #PWR0235
 U 1 1 5D483C15
 P 1400 5600
@@
 Connection ~ 1400 5600
 $Comp
-L pcb-rescue:C-Device-pcb-rescue C?
+L Device:C C?
 U 1 1 5D489120
 P 1400 7450
@@
 $EndComp
 $Comp
-L pcb-rescue:GND-power-pcb-rescue #PWR?
+L power:GND #PWR?
 U 1 1 5D489128
 P 1400 7600
@@
 $EndComp
 $Comp
-L pcb-rescue:Conn_01x18-Connector_Generic-pcb-rescue J500
+L Connector_Generic:Conn_01x18 J500
 U 1 1 5D4BB38B
 P 9600 1600
@@
 $EndComp
 $Comp
-L pcb-rescue:GND-power-pcb-rescue #PWR0237
+L power:GND #PWR0237
 U 1 1 5D4BF290
 P 9300 2500
@@
 Connection ~ 4500 6100
 $Comp
-L pcb-rescue:C-Device-pcb-rescue C508
+L Device:C C508
 U 1 1 5D5F56B0
 P 4250 6100
@@
 $EndComp
 $Comp
-L pcb-rescue:GND-power-pcb-rescue #PWR0238
+L power:GND #PWR0238
 U 1 1 5D5FB1D3
 P 4000 6100
@@
 	4000 6100 4100 6100
 $Comp
-L pcb-rescue:+3V3-power-pcb-rescue #PWR?
+L power:+3V3 #PWR?
 U 1 1 5D622DCE
 P 5400 4600
@@
 $EndComp
 $Comp
-L pcb-rescue:IRLML6402-Transistor_FET-pcb-rescue Q?
+L Transistor_FET:IRLML6402 Q?
 U 1 1 5D622DD4
 P 5300 4900
@@
 	5400 4600 5400 4700
 $Comp
-L pcb-rescue:R-Device-pcb-rescue R?
+L Device:R R?
 U 1 1 5D622DDB
 P 4900 5150
@@
 $EndComp
 $Comp
-L pcb-rescue:R-Device-pcb-rescue R?
+L Device:R R?
 U 1 1 5D622DE1
 P 4900 4650
@@
 	4900 5000 4900 4900
 $Comp
-L pcb-rescue:GND-power-pcb-rescue #PWR?
+L power:GND #PWR?
 U 1 1 5D622DED
 P 4900 5300
@@
 $EndComp
 $Comp
-L pcb-rescue:+3V3-power-pcb-rescue #PWR?
+L power:+3V3 #PWR?
 U 1 1 5D622DF3
 P 4900 4500
@@
 $EndComp
 $Comp
-L pcb-rescue:D_Schottky-Device-pcb-rescue D?
+L Device:D_Schottky D?
 U 1 1 5D622DF9
 P 4650 4900
@@
 NoConn ~ 4600 6500
 $Comp
-L pcb-rescue:R-Device-pcb-rescue R502
+L Device:R R502
 U 1 1 5D672E77
 P 4350 6700
@@
 $EndComp
 $Comp
-L pcb-rescue:C-Device-pcb-rescue C509
+L Device:C C509
 U 1 1 5D673908
 P 3950 6700
@@
 $EndComp
 $Comp
-L pcb-rescue:C-Device-pcb-rescue C510
+L Device:C C510
 U 1 1 5D674718
 P 4300 7050
@@
 $EndComp
 $Comp
-L pcb-rescue:C-Device-pcb-rescue C511
+L Device:C C511
 U 1 1 5D6756DB
 P 6150 5600
@@
 $EndComp
 $Comp
-L pcb-rescue:R-Device-pcb-rescue R503
+L Device:R R503
 U 1 1 5D675D3D
 P 5800 6250
@@
 $EndComp
 $Comp
-L pcb-rescue:R-Device-pcb-rescue R509
+L Device:R R509
 U 1 1 5D67C719
 P 6150 6400
@@
 $EndComp
 $Comp
-L pcb-rescue:C-Device-pcb-rescue C512
+L Device:C C512
 U 1 1 5D67D52C
 P 6400 6850
@@
 $EndComp
 $Comp
-L pcb-rescue:D_Schottky-Device-pcb-rescue D501
+L Device:D_Schottky D501
 U 1 1 5D685CDF
 P 6150 6600
@@
 	6000 6600 5800 6600
 $Comp
-L pcb-rescue:GND-power-pcb-rescue #PWR?
+L power:GND #PWR?
 U 1 1 5D6AFE75
 P 6400 5600
@@
 	6300 5600 6400 5600
 $Comp
-L pcb-rescue:GND-power-pcb-rescue #PWR?
+L power:GND #PWR?
 U 1 1 5D6B732F
 P 6400 7000
@@
 $EndComp
 $Comp
-L pcb-rescue:GND-power-pcb-rescue #PWR?
+L power:GND #PWR?
 U 1 1 5D6B76FB
 P 5600 7200
@@
 $EndComp
 $Comp
-L pcb-rescue:GND-power-pcb-rescue #PWR?
+L power:GND #PWR?
 U 1 1 5D6B7A0D
 P 4600 7200
@@
 $EndComp
 $Comp
-L pcb-rescue:GND-power-pcb-rescue #PWR?
+L power:GND #PWR?
 U 1 1 5D6B80FB
 P 3800 6700
@@
 $EndComp
 $Comp
-L pcb-rescue:GND-power-pcb-rescue #PWR?
+L power:GND #PWR?
 U 1 1 5D6B8450
 P 4300 7200
@@
 NoConn ~ 5600 6800
 $Comp
-L pcb-rescue:L-Device-pcb-rescue L500
+L Device:L_Small L500
 U 1 1 5D6F546B
 P 5800 6850
@@
 $EndComp
 $Comp
-L pcb-rescue:GND-power-pcb-rescue #PWR?
+L power:GND #PWR?
 U 1 1 5D6F67EF
 P 5800 7100
@@
 Connection ~ 6400 6400
 $Comp
-L pcb-rescue:R_POT-Device-pcb-rescue RV500
+L Device:R_POT RV500
 U 1 1 5D72C05F
 P 5800 5800
@@
 	7200 6000 7200 6050
 $Comp
-L pcb-rescue:R-Device-pcb-rescue R504
+L Device:R R504
 U 1 1 5D585916
 P 7200 6250
@@
 	6700 5750 6700 6400
 $Comp
-L pcb-rescue:LM324-Amplifier_Operational-pcb-rescue U502
+L Amplifier_Operational:LM324 U502
 U 5 1 5D80D00D
 P 6800 5450
@@
 	7800 5050 7800 5150
 $Comp
-L pcb-rescue:LM324-Amplifier_Operational-pcb-rescue U502
+L Amplifier_Operational:LM324 U502
 U 4 1 5D78D689
 P 8100 6150
@@
 $EndComp
 $Comp
-L pcb-rescue:LM324-Amplifier_Operational-pcb-rescue U502
+L Amplifier_Operational:LM324 U502
 U 3 1 5D78AB11
 P 8100 5750
@@
 $EndComp
 $Comp
-L pcb-rescue:LM324-Amplifier_Operational-pcb-rescue U502
+L Amplifier_Operational:LM324 U502
 U 2 1 5D787DB9
 P 8100 5350
@@
 $EndComp
 $Comp
-L pcb-rescue:LM324-Amplifier_Operational-pcb-rescue U502
+L Amplifier_Operational:LM324 U502
 U 1 1 5D783130
 P 8100 4950
@@
 	7200 5700 7200 5650
 $Comp
-L pcb-rescue:R-Device-pcb-rescue R508
+L Device:R R508
 U 1 1 5D7560C1
 P 7200 4650
@@
 $EndComp
 $Comp
-L pcb-rescue:R-Device-pcb-rescue R507
+L Device:R R507
 U 1 1 5D755DDC
 P 7200 5050
@@
 $EndComp
 $Comp
-L pcb-rescue:R-Device-pcb-rescue R505
+L Device:R R505
 U 1 1 5D753D04
 P 7200 5850
@@
 -11.6V to -17.8V
 $Comp
-L pcb-rescue:R-Device-pcb-rescue R506
+L Device:R R506
 U 1 1 5D75597D
 P 7200 5450
@@
 $EndComp
 $Comp
-L pcb-rescue:+1V8-power-pcb-rescue #PWR0224
+L power:+1V8 #PWR0224
 U 1 1 5D45A159
 P 5400 2800
@@
 $EndComp
 $Comp
-L pcb-rescue:+3V3-power-pcb-rescue #PWR0225
+L power:+3V3 #PWR0225
 U 1 1 5D45AD93
 P 4600 2800
@@
 	5400 3000 5400 2800
 $Comp
-L pcb-rescue:C-Device-pcb-rescue C500
+L Device:C C500
 U 1 1 5D4632AC
 P 5400 3450
@@
 $EndComp
 $Comp
-L pcb-rescue:C-Device-pcb-rescue C501
+L Device:C C501
 U 1 1 5D463E9F
 P 5000 3450
@@
 $EndComp
 $Comp
-L pcb-rescue:C-Device-pcb-rescue C502
+L Device:C C502
 U 1 1 5D46402C
 P 4600 3450
@@
 $EndComp
 $Comp
-L pcb-rescue:C-Device-pcb-rescue C503
+L Device:C C503
 U 1 1 5D464243
 P 4200 3450
@@
 $EndComp
 $Comp
-L pcb-rescue:GND-power-pcb-rescue #PWR0226
+L power:GND #PWR0226
 U 1 1 5D468CD4
 P 5400 3600
@@
 $EndComp
 $Comp
-L pcb-rescue:GND-power-pcb-rescue #PWR0227
+L power:GND #PWR0227
 U 1 1 5D46903A
 P 5000 3600
@@
 $EndComp
 $Comp
-L pcb-rescue:GND-power-pcb-rescue #PWR0228
+L power:GND #PWR0228
 U 1 1 5D46925D
 P 4600 3600
@@
 $EndComp
 $Comp
-L pcb-rescue:GND-power-pcb-rescue #PWR0229
+L power:GND #PWR0229
 U 1 1 5D4694F7
 P 4200 3600
@@
 	7300 2000 7700 2000
 $Comp
-L pcb-rescue:R_Pack04-Device-pcb-rescue RN502
+L Device:R_Pack04 RN502
 U 1 1 5D42A1C4
 P 7100 1600

Commit message: pcb: bug fixes
Parts:
- removed C509: 68nF, Capacitor_SMD:C_0402_1005Metric, symbol Device:C
- removed C511: 1uF, Capacitor_SMD:C_0402_1005Metric, symbol Device:C
- removed D500: RB521S30T1G, Diode_SMD:D_SOD-523, symbol Device:D_Schottky
- removed Q500: IRLML6402, Package_TO_SOT_SMD:SOT-23, symbol Transistor_FET:IRLML6402
- removed R500: 100K, Resistor_SMD:R_0603_1608Metric, symbol Device:R
- removed R502: 15K, Resistor_SMD:R_0603_1608Metric, symbol Device:R
- removed U501: ADP5075, footprints:WLCSP-12_3x4, symbol symbols:ADP5075
- added L501: 22uH, Inductor_SMD:L_Vishay_IHLP-1212, symbol Device:L
- added U501: LT1617, Package_TO_SOT_SMD:TSOT-23-5, symbol symbols:LT1617
- C510: value 10uF -> 220nF
- D501: value DFLS240 -> MBR0530
- L500: value 15uH -> 22uH; symbol Device:L_Small -> Device:L
- R503: value 100K -> 330K
- R509: value 2.32M -> 20K
- RV500: value RK14J11A0A02 -> RK14J11A0A02/50K
Connections:
- net labels removed: +3V3_LCD
- wire segments 210 -> 189
- no-connect marks 31 -> 29
Other:
- note added: "-7V to -22V"
- note removed: "-11.6V to -17.8V"
- moved on the sheet: C508, C510, C512, D501, L500, R501, R503, R504, R505, R506, R507, R508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
