File: pcb/power.sch (KiCad schematic (older format))
At the start: 69 parts, among them SW1 SW_SP3T, U1 LTC3456, U100 MCIMX7S5EVM08SC, U2 LTC3549, U3 LTC3549

Commit message: pcb: routing
Parts:
- BT1: footprint Battery:BatteryHolder_Keystone_2468_2xAAA -> footprints:BatteryHolder_Keystone_5201_5223; symbol Device:Battery -> pcb-rescue:Battery-Device
- BT_Backup1: symbol Device:Battery_Cell -> pcb-rescue:Battery_Cell-Device
- C1, C10, C11, C12, C13, C14, C15, C16, C17, C18, C19, C2, C20, C21, C22, C23, C24, C25, C26, C27, C28, C29, C3, C30, C31, C33, C34, C35, C36, C37, C38, C39, C4, C40, C41, C5, C6, C7, C8, C9: symbol Device:C -> pcb-rescue:C-Device
- D1, D2: symbol Device:D_Shockley -> pcb-rescue:D_Shockley-Device
- D3: symbol Device:LED -> pcb-rescue:LED-Device
- L1, L2, L3, L4, L5, L6: symbol Device:L -> pcb-rescue:L-Device
- R1, R10, R11, R12, R13, R2, R3, R4, R5, R6, R7, R8, R9: symbol Device:R -> pcb-rescue:R-Device
- SW1: symbol Switch:SW_SP3T -> pcb-rescue:SW_SP3T-Switch
Connections:
- wire segments 208 -> 209

Commit message: pcb: rev 0.1
Parts:
- added C42: 100uF, Capacitor_SMD:C_Elec_5x5.4, symbol Device:CP
- BT1: symbol pcb-rescue:Battery-Device -> pcb-rescue:Battery-Device-pcb-rescue
- BT_Backup1: symbol pcb-rescue:Battery_Cell-Device -> pcb-rescue:Battery_Cell-Device-pcb-rescue
- C1, C10, C11, C12, C13, C14, C15, C16, C17, C18, C19, C20, C21, C22, C23, C24, C25, C26, C27, C28, C29, C3, C30, C31, C33, C34, C35, C36, C37, C38, C39, C4, C40, C41, C5, C6, C8, C9: symbol pcb-rescue:C-Device -> pcb-rescue:C-Device-pcb-rescue
- C2, C7: value 10uF -> 100uF; footprint Capacitor_SMD:C_0603_1608Metric -> Capacitor_SMD:C_1206_3216Metric; symbol pcb-rescue:C-Device -> pcb-rescue:C-Device-pcb-rescue
- D1, D2: symbol pcb-rescue:D_Shockley-Device -> pcb-rescue:D_Schottky-Device-pcb-rescue
- D3: symbol pcb-rescue:LED-Device -> pcb-rescue:LED-Device-pcb-rescue
- L1, L2, L3, L4, L5, L6: symbol pcb-rescue:L-Device -> pcb-rescue:L-Device-pcb-rescue
- R1, R10, R11, R13, R2, R3, R5, R6, R8, R9: symbol pcb-rescue:R-Device -> pcb-rescue:R-Device-pcb-rescue
- R12, R4, R7: footprint Resistor_SMD:R_1210_3225Metric -> Resistor_SMD:R_1206_3216Metric; symbol pcb-rescue:R-Device -> pcb-rescue:R-Device-pcb-rescue
- SW1: symbol pcb-rescue:SW_SP3T-Switch -> pcb-rescue:SW_SP3T-Switch-pcb-rescue
Connections:
- net +BATT: now also C42.1
- net GND: now also C42.2
- net +RTC: now reaches D1.1 (K), D2.1 (K), U100.AD8 (VDD_SNVS_IN)
