File: pcb/power.sch (KiCad schematic (older format))
At the start: 70 parts, among them SW1 SW_SP3T, U1 LTC3456, U100 MCIMX7S5EVM08SC, U2 LTC3549, U3 LTC3549

Commit message: pcb: remap schematic symbols
Parts:
- BT1: symbol pcb-rescue:Battery-Device-pcb-rescue -> Device:Battery
- BT_Backup1: symbol pcb-rescue:Battery_Cell-Device-pcb-rescue -> Device:Battery_Cell
- C1, C10, C11, C12, C13, C14, C15, C16, C17, C18, C19, C2, C20, C21, C22, C23, C24, C25, C26, C27, C28, C29, C3, C30, C31, C33, C34, C35, C36, C37, C38, C39, C4, C40, C41, C5, C6, C7, C8, C9: symbol pcb-rescue:C-Device-pcb-rescue -> Device:C
- D1, D2: symbol pcb-rescue:D_Schottky-Device-pcb-rescue -> Device:D_Schottky
- D3: symbol pcb-rescue:LED-Device-pcb-rescue -> Device:LED
- L1, L2, L3, L4, L5, L6: symbol pcb-rescue:L-Device-pcb-rescue -> Device:L_Small
- R1, R10, R11, R12, R13, R2, R3, R4, R5, R6, R7, R8, R9: symbol pcb-rescue:R-Device-pcb-rescue -> Device:R
- SW1: symbol pcb-rescue:SW_SP3T-Switch-pcb-rescue -> Switch:SW_SP3T

Commit message: pcb: bug fixes
Parts:
- BT1: footprint footprints:BatteryHolder_Keystone_5201_5223 -> footprints:BatteryHolder_Keystone_5204_5226
- C12, C9: value 220pF -> 22pF
- L1, L2, L3, L4, L5, L6: symbol Device:L_Small -> Device:L
Changed lines of the file:
@@
 F 0 "BT1" H 1708 4896 50  0000 L CNN
 F 1 "Battery" H 1708 4805 50  0000 L CNN
-F 2 "footprints:BatteryHolder_Keystone_5201_5223" V 1600 4910 50  0001 C CNN
+F 2 "footprints:BatteryHolder_Keystone_5204_5226" V 1600 4910 50  0001 C CNN
 F 3 "~" V 1600 4910 50  0001 C CNN
 	1    1600 4850
@@
 Connection ~ 2300 4650
 $Comp
-L Device:L_Small L1
+L Device:L L1
 U 1 1 5D2F2270
 P 2950 5350
@@
 $EndComp
 $Comp
-L Device:L_Small L3
+L Device:L L3
 U 1 1 5D311C05
 P 5000 5000
@@
 $EndComp
 $Comp
-L Device:L_Small L2
+L Device:L L2
 U 1 1 5D312A2A
 P 4700 4800
@@
 Wire Wire Line
 	4600 5150 5000 5150
-Wire Wire Line
-	4600 4850 5000 4850
 $Comp
 L Device:C C6
@@
 	1    0    0    -1
 $EndComp
-Wire Wire Line
-	5400 4850 5000 4850
-Connection ~ 5000 4850
 Wire Wire Line
 	5800 4750 4600 4750
@@
 	6000 1900 6000 2000
 $Comp
-L Device:L_Small L5
+L Device:L L5
 U 1 1 5D330C85
 P 7050 1700
@@
 P 7700 1850
 F 0 "C12" H 7815 1896 50  0000 L CNN
-F 1 "220pF" H 7815 1805 50  0000 L CNN
+F 1 "22pF" H 7815 1805 50  0000 L CNN
 F 2 "Capacitor_SMD:C_0402_1005Metric" H 7738 1700 50  0001 C CNN
 F 3 "~" H 7700 1850 50  0001 C CNN
@@
 	2400 1900 2400 2000
 $Comp
-L Device:L_Small L4
+L Device:L L4
 U 1 1 5D474768
 P 3450 1700
@@
 P 4100 1850
 F 0 "C9" H 4215 1896 50  0000 L CNN
-F 1 "220pF" H 4215 1805 50  0000 L CNN
+F 1 "22pF" H 4215 1805 50  0000 L CNN
 F 2 "Capacitor_SMD:C_0402_1005Metric" H 4138 1700 50  0001 C CNN
 F 3 "~" H 4100 1850 50  0001 C CNN
@@
 Connection ~ 6600 4150
 $Comp
-L Device:L_Small L6
+L Device:L L6
 U 1 1 5D5F1F4C
 P 7250 4900
@@
 Wire Wire Line
 	7100 5400 8900 5400
+Wire Wire Line
+	4600 4850 5000 4850
+Connection ~ 5000 4850
+Wire Wire Line
+	5000 4850 5400 4850
 $EndSCHEMATC
