File: pcb/storage.sch (KiCad schematic (older format))
At the start: 10 parts, among them U100 MCIMX7S5EVM08SC

Commit message: pcb: working on sch
Parts:
- added C303, C312: 4.7uF, symbol Device:C
- added C304, C311, C313: 100nF, symbol Device:C
- added C305: 2.2uF, symbol Device:C
- added C306, C307, C308, C309: 220nF, symbol Device:C
- added C310: 10uF, symbol Device:C
- added D300: RB521S30T1G, symbol Device:D_Schottky
- added Q302: 2SK3018, symbol Device:Q_NMOS_SGD
- added Q?: IRLML6402, Package_TO_SOT_SMD:SOT-23, symbol Transistor_FET:IRLML6402
- added R304, R308: 100K, symbol Device:R
- added R305: 10K, symbol Device:R
- added R306: 560K/1%, symbol Device:R
- added R307: 100K/1%, symbol Device:R
- added R309: 487K/1%, symbol Device:R
- added U300: ADP123, Package_TO_SOT_SMD:TSOT-23-5, symbol Regulator_Linear:ADP7142AUZJ
- gave numbers to parts that had none: 1
Connections:
- net +3V3: now also U100.F12 (NVCC_SAI), U100.H8 (NVCC_SD2), U100.K8 (NVCC_SD3), C306.1, C308.1, C309.1, C310.1, C311.1, Q?.2 (S), R304.1, U300.1 (VIN), U300.3 (EN); no longer C301.1, C302.1, MICRO_SD.4 (VDD)
- net GND: now also U301.4 (GND), C303.2, C304.2, C305.2, C306.2, C307.2, C308.2, C309.2, C310.2, C311.2, C312.2, C313.2, R305.2, R307.2, R308.2, U300.2 (GND)
- net at U100.E7 (NVCC_SD1): now also R301.1, R302.1, C307.1, C312.1, C313.1, R306.1, R309.1, U300.5 (VOUT)
- net at U100.J9 (PVCC_SAI_SD_CAP): now also C305.1
- net ~QSPI_SS0: now reaches U301.1 (#CS)
- net ~QSPI_SS0: now also R300.2
- net QSPI_D1: now reaches U301.2 (DO(IO1))
- net QSPI_D2: now reaches U301.3 (#WP(IO2))
- net QSPI_D0: now reaches U301.5 (DI(IO0))
- net QSPI_SCLK: now reaches U301.6 (CLK)
- net QSPI_D3: now reaches U301.7 (#HOLD(IO3))
- net +1V8: now reaches U301.8 (VCC)
- net +1V8: now also R300.1, C303.1, C304.1
- new net: D300.1 (K), Q?.1 (G), R304.2, R305.1
- new net: C301.1, C302.1, MICRO_SD.4 (VDD), Q?.3 (D)
- new net: Q302.1 (S), R306.2, R307.1, U300.4 (FB)
- new net: Q302.3 (D), R309.2
- new net PMIC_STBY_REQ: D300.2 (A)
- new net SD1_VSELECT: Q302.2 (G), R308.1
- no-connect marks 0 -> 17
Other:
- note added: "47uF is required to comply with SD 3.0 spec"
- note added: "FB = 0.5V, use 560K/487K/100K\nFB = 0.8V, use 499K/330K/160K\nFB = 1.0V, use 464K/243K/200K"
- moved on the sheet: C300, C301, C302, MICRO_SD, R300, R301, R302, R303, U100F, U301

Commit message: pcb: draw sch for wifi & bt
Connections:
- net PMIC_STBY_REQ renamed SD_PWR_EN
Changed lines of the file:
@@
 $Descr A4 11693 8268
 encoding utf-8
-Sheet 5 10
+Sheet 5 11
 Title "SPI Flash & TF-Card"
 Date ""
@@
 $EndComp
 Text GLabel 7100 2100 0    50   Input ~ 0
-PMIC_STBY_REQ
+SD_PWR_EN
 Wire Wire Line
 	8100 2300 8100 2700

Commit message: pcb: working on sch
Connections:
- net CCM_CLKO2: now reaches U100.C4 (SD1_WP)
- no-connect marks 17 -> 16
Other:
- note added: "Configure as 32kHz clock output"
Changed lines of the file:
@@
 Wire Wire Line
 	7100 2100 7200 2100
-NoConn ~ 4400 4600
 NoConn ~ 4400 4700
 NoConn ~ 4400 5500
@@
 Wire Wire Line
 	8400 5000 8400 5100
+Text GLabel 4600 4600 2    50   Output ~ 0
+CCM_CLKO2
+Wire Wire Line
+	4400 4600 4600 4600
+Text Notes 5900 4800 2    50   ~ 0
+Configure as 32kHz clock output
 $EndSCHEMATC

Commit message: pcb: finishing sch for r0.1
Parts:
- C300, C302, C304, C305, C306, C307, C308, C309, C311, C313: footprint (none) -> Capacitor_SMD:C_0402_1005Metric
- C301: footprint (none) -> Capacitor_SMD:C_0805_2012Metric
- C303, C310, C312: footprint (none) -> Capacitor_SMD:C_0603_1608Metric
- D300: footprint (none) -> Diode_SMD:D_SOD-523
- MICRO_SD300: renamed from MICRO_SD; footprint (none) -> footprints:TFC-WPAPR-08
- Q302: footprint (none) -> Package_TO_SOT_SMD:SOT-23
- R300, R301, R302, R303, R304, R305, R306, R307, R308, R309: footprint (none) -> Resistor_SMD:R_0603_1608Metric
- U100: footprint (none) -> footprints:BGA-541_25x25_19.0x19.0mm
- U301: footprint (none) -> Package_SON:WSON-8-1EP_6x5mm_P1.27mm_EP3.4x4mm
- gave numbers to parts that had none: 1
Connections:
- net +1V8: now also C306.1, U100.F12 (NVCC_SAI)
- net +3V3: no longer C306.1, U100.F12 (NVCC_SAI)
- net SAI2_RXD: no longer names the net of U100.E9 (SAI2_RXD)
- net SAI2_TXC: no longer names the net of U100.D8 (SAI2_TXC)
- net SAI2_TXD: no longer names the net of U100.E8 (SAI2_TXD)
- net SAI2_TXFS: no longer names the net of U100.D9 (SAI2_TXFS)
- net SD_PWR_EN renamed ~SD_PWR_EN
- no-connect marks 16 -> 23

Commit message: pcb: routing
Parts:
- C300, C301, C302, C303, C304, C305, C306, C307, C308, C309, C310, C311, C312, C313: symbol Device:C -> pcb-rescue:C-Device
- D300: symbol Device:D_Schottky -> pcb-rescue:D_Schottky-Device
- Q300: symbol Transistor_FET:IRLML6402 -> pcb-rescue:IRLML6402-Transistor_FET
- Q302: symbol Device:Q_NMOS_SGD -> pcb-rescue:Q_NMOS_SGD-Device
- R300, R301, R302, R303, R304, R305, R306, R307, R308, R309: symbol Device:R -> pcb-rescue:R-Device
- U300: symbol Regulator_Linear:ADP7142AUZJ -> pcb-rescue:ADP7142AUZJ-Regulator_Linear
Changed lines of the file:
@@
 	6900 3700 7400 3700
 $Comp
-L power:GND #PWR0200
+L pcb-rescue:GND-power #PWR0200
 U 1 1 5DBA2B48
 P 7300 4300
@@
 To Audio DAC\n
 $Comp
-L Device:R R300
+L pcb-rescue:R-Device R300
 U 1 1 5DBBE698
 P 7150 5350
@@
 $EndComp
 $Comp
-L Device:R R301
+L pcb-rescue:R-Device R301
 U 1 1 5DBC08BA
 P 6400 2950
@@
 $EndComp
 $Comp
-L Device:R R302
+L pcb-rescue:R-Device R302
 U 1 1 5DBC0C88
 P 5900 2950
@@
 $EndComp
 $Comp
-L Device:R R303
+L pcb-rescue:R-Device R303
 U 1 1 5DBC2BE9
 P 6650 3700
@@
 	5900 2800 5900 2700
 $Comp
-L Device:C C300
+L pcb-rescue:C-Device C300
 U 1 1 5DBD27EC
 P 6900 4350
@@
 $EndComp
 $Comp
-L power:GND #PWR0201
+L pcb-rescue:GND-power #PWR0201
 U 1 1 5DBD7168
 P 6900 4600
@@
 	6900 4500 6900 4600
 $Comp
-L Device:C C301
+L pcb-rescue:C-Device C301
 U 1 1 5DBD9F72
 P 7700 2850
@@
 $EndComp
 $Comp
-L Device:C C302
+L pcb-rescue:C-Device C302
 U 1 1 5DBDAEE7
 P 8100 2850
@@
 $EndComp
 $Comp
-L power:GND #PWR0202
+L pcb-rescue:GND-power #PWR0202
 U 1 1 5DBDB16E
 P 7700 3000
@@
 Connection ~ 7700 2700
 $Comp
-L power:+3V3 #PWR0203
+L pcb-rescue:+3V3-power #PWR0203
 U 1 1 5D1E3230
 P 8100 1800
@@
 $EndComp
 $Comp
-L Transistor_FET:IRLML6402 Q300
+L pcb-rescue:IRLML6402-Transistor_FET Q300
 U 1 1 5D1E5978
 P 8000 2100
@@
 	7150 5100 8400 5100
 $Comp
-L Device:R R305
+L pcb-rescue:R-Device R305
 U 1 1 5D1FE40C
 P 7600 2350
@@
 $EndComp
 $Comp
-L Device:R R304
+L pcb-rescue:R-Device R304
 U 1 1 5D1FF47A
 P 7600 1850
@@
 	7600 2200 7600 2100
 $Comp
-L power:GND #PWR0204
+L pcb-rescue:GND-power #PWR0204
 U 1 1 5D20AD53
 P 7600 2500
@@
 $EndComp
 $Comp
-L power:+3V3 #PWR0205
+L pcb-rescue:+3V3-power #PWR0205
 U 1 1 5D20B20B
 P 7600 1700
@@
 $EndComp
 $Comp
-L Device:D_Schottky D300
+L pcb-rescue:D_Schottky-Device D300
 U 1 1 5D20C1D1
 P 7350 2100
@@
 	7150 5200 7150 5100
 $Comp
-L power:GND #PWR0206
+L pcb-rescue:GND-power #PWR0206
 U 1 1 5D24A79B
 P 8400 6200
@@
 	8400 6100 8400 6200
 $Comp
-L Device:C C303
+L pcb-rescue:C-Device C303
 U 1 1 5D24DBD3
 P 8800 5250
@@
 $EndComp
 $Comp
-L Device:C C304
+L pcb-rescue:C-Device C304
 U 1 1 5D24DBD9
 P 9200 5250
@@
 $EndComp
 $Comp
-L power:GND #PWR0207
+L pcb-rescue:GND-power #PWR0207
 U 1 1 5D24DBDF
 P 8800 5400
@@
 	7500 2100 7600 2100
 $Comp
-L Device:C C305
+L pcb-rescue:C-Device C305
 U 1 1 5D259DFD
 P 2600 7250
@@
 	2600 7000 2600 7100
 $Comp
-L power:GND #PWR0208
+L pcb-rescue:GND-power #PWR0208
 U 1 1 5D25D3D4
 P 2600 7400
@@
 $EndComp
 $Comp
-L Device:C C306
+L pcb-rescue:C-Device C306
 U 1 1 5D25F58F
 P 2600 2650
@@
 $EndComp
 $Comp
-L power:GND #PWR0209
+L pcb-rescue:GND-power #PWR0209
 U 1 1 5D2600DE
 P 2600 2900
@@
 	2600 2900 2600 2800
 $Comp
-L power:+3V3 #PWR0210
+L pcb-rescue:+3V3-power #PWR0210
 U 1 1 5D2689FB
 P 2600 4900
@@
 $EndComp
 $Comp
-L Device:C C308
+L pcb-rescue:C-Device C308
 U 1 1 5D268A01
 P 2600 5250
@@
 $EndComp
 $Comp
-L power:GND #PWR0211
+L pcb-rescue:GND-power #PWR0211
 U 1 1 5D268A07
 P 2600 5500
@@
 	2600 5500 2600 5400
 $Comp
-L power:+3V3 #PWR0212
+L pcb-rescue:+3V3-power #PWR0212
 U 1 1 5D26D067
 P 2600 5900
@@
 $EndComp
 $Comp
-L Device:C C309
+L pcb-rescue:C-Device C309
 U 1 1 5D26D06D
 P 2600 6250
@@
 $EndComp
 $Comp
-L power:GND #PWR0213
+L pcb-rescue:GND-power #PWR0213
 U 1 1 5D26D073
 P 2600 6500
@@
 Connection ~ 2600 5900
 $Comp
-L Device:C C307
+L pcb-rescue:C-Device C307
 U 1 1 5D273248
 P 2600 4250
@@
 $EndComp
 $Comp
-L power:GND #PWR0214
+L pcb-rescue:GND-power #PWR0214
 U 1 1 5D27324E
 P 2600 4500
@@
 	2600 4500 2600 4400
 $Comp
-L Regulator_Linear:ADP7142AUZJ U300
+L pcb-rescue:ADP7142AUZJ-Regulator_Linear U300
 U 1 1 5D27B732
 P 3800 1000
@@
 Connection ~ 6400 4100
 $Comp
-L power:GND #PWR0215
+L pcb-rescue:GND-power #PWR0215
 U 1 1 5D39B0B3
 P 3800 1300
@@
 $EndComp
 $Comp
-L Device:C C310
+L pcb-rescue:C-Device C310
 U 1 1 5D39B62C
 P 2500 1050
@@
 $EndComp
 $Comp
-L Device:C C311
+L pcb-rescue:C-Device C311
 U 1 1 5D39C092
 P 2900 1050
@@
 $EndComp
 $Comp
-L Device:Q_NMOS_SGD Q302
+L pcb-rescue:Q_NMOS_SGD-Device Q302
 U 1 1 5D3A2E7B
 P 4900 1300
@@
 $EndComp
 $Comp
-L Device:R R307
+L pcb-rescue:R-Device R307
 U 1 1 5D3AB9EC
 P 4400 1350
@@
 $EndComp
 $Comp
-L Device:R R306
+L pcb-rescue:R-Device R306
 U 1 1 5D3ABE8A
 P 4400 1050
@@
 $EndComp
 $Comp
-L Device:R R308
+L pcb-rescue:R-Device R308
 U 1 1 5D3AF41C
 P 4900 1650
@@
 $EndComp
 $Comp
-L Device:R R309
+L pcb-rescue:R-Device R309
 U 1 1 5D3BF697
 P 5200 1050
@@
 $EndComp
 $Comp
-L Device:C C312
+L pcb-rescue:C-Device C312
 U 1 1 5D3C0823
 P 5600 1050
@@
 $EndComp
 $Comp
-L Device:C C313
+L pcb-rescue:C-Device C313
 U 1 1 5D3C0829
 P 6000 1050
@@
 $EndComp
 $Comp
-L power:GND #PWR0216
+L pcb-rescue:GND-power #PWR0216
 U 1 1 5D3C082F
 P 5600 1200
@@
 Connection ~ 5600 1200
 $Comp
-L power:GND #PWR0217
+L pcb-rescue:GND-power #PWR0217
 U 1 1 5D3CF6CC
 P 4900 1800
@@
 $EndComp
 $Comp
-L power:GND #PWR0218
+L pcb-rescue:GND-power #PWR0218
 U 1 1 5D3CFB51
 P 4400 1500
@@
 	2900 1200 2500 1200
 $Comp
-L power:GND #PWR0219
+L pcb-rescue:GND-power #PWR0219
 U 1 1 5D3FB2DA
 P 2500 1200
@@
 Connection ~ 2500 1200
 $Comp
-L power:+3V3 #PWR0220
+L pcb-rescue:+3V3-power #PWR0220
 U 1 1 5D3FB6DC
 P 2500 900
@@
 FB = 0.5V, use 560K/487K/100K\nFB = 0.8V, use 499K/330K/160K\nFB = 1.0V, use 464K/243K/200K
 $Comp
-L power:+1V8 #PWR0221
+L pcb-rescue:+1V8-power #PWR0221
 U 1 1 5D3F1E82
 P 8400 5000
@@
 Configure as 32kHz clock output
 $Comp
-L power:+1V8 #PWR0222
+L pcb-rescue:+1V8-power #PWR0222
 U 1 1 5D2012F3
 P 2600 2300

Commit message: pcb: rev 0.1
Parts:
- C300, C301, C302, C303, C304, C305, C306, C307, C308, C309, C310, C311, C312, C313: symbol pcb-rescue:C-Device -> pcb-rescue:C-Device-pcb-rescue
- D300: symbol pcb-rescue:D_Schottky-Device -> pcb-rescue:D_Schottky-Device-pcb-rescue
- Q300: symbol pcb-rescue:IRLML6402-Transistor_FET -> pcb-rescue:IRLML6402-Transistor_FET-pcb-rescue
- Q302: symbol pcb-rescue:Q_NMOS_SGD-Device -> pcb-rescue:Q_NMOS_SGD-Device-pcb-rescue
- R300, R301, R302, R303, R304, R305, R306, R307, R308, R309: symbol pcb-rescue:R-Device -> pcb-rescue:R-Device-pcb-rescue
- U300: symbol pcb-rescue:ADP7142AUZJ-Regulator_Linear -> pcb-rescue:ADP7142AUZJ-Regulator_Linear-pcb-rescue
Changed lines of the file:
@@
 encoding utf-8
 Sheet 5 11
-Title "SPI Flash & TF-Card"
-Date ""
+Title "RhythmPocket"
+Date "2019-07-16"
 Rev "R0.1"
 Comp "ZephRay"
@@
 	6900 3700 7400 3700
 $Comp
-L pcb-rescue:GND-power #PWR0200
+L pcb-rescue:GND-power-pcb-rescue #PWR0200
 U 1 1 5DBA2B48
 P 7300 4300
@@
 To Audio DAC\n
 $Comp
-L pcb-rescue:R-Device R300
+L pcb-rescue:R-Device-pcb-rescue R300
 U 1 1 5DBBE698
 P 7150 5350
@@
 $EndComp
 $Comp
-L pcb-rescue:R-Device R301
+L pcb-rescue:R-Device-pcb-rescue R301
 U 1 1 5DBC08BA
 P 6400 2950
@@
 $EndComp
 $Comp
-L pcb-rescue:R-Device R302
+L pcb-rescue:R-Device-pcb-rescue R302
 U 1 1 5DBC0C88
 P 5900 2950
@@
 $EndComp
 $Comp
-L pcb-rescue:R-Device R303
+L pcb-rescue:R-Device-pcb-rescue R303
 U 1 1 5DBC2BE9
 P 6650 3700
@@
 	5900 2800 5900 2700
 $Comp
-L pcb-rescue:C-Device C300
+L pcb-rescue:C-Device-pcb-rescue C300
 U 1 1 5DBD27EC
 P 6900 4350
@@
 $EndComp
 $Comp
-L pcb-rescue:GND-power #PWR0201
+L pcb-rescue:GND-power-pcb-rescue #PWR0201
 U 1 1 5DBD7168
 P 6900 4600
@@
 	6900 4500 6900 4600
 $Comp
-L pcb-rescue:C-Device C301
+L pcb-rescue:C-Device-pcb-rescue C301
 U 1 1 5DBD9F72
 P 7700 2850
@@
 $EndComp
 $Comp
-L pcb-rescue:C-Device C302
+L pcb-rescue:C-Device-pcb-rescue C302
 U 1 1 5DBDAEE7
 P 8100 2850
@@
 $EndComp
 $Comp
-L pcb-rescue:GND-power #PWR0202
+L pcb-rescue:GND-power-pcb-rescue #PWR0202
 U 1 1 5DBDB16E
 P 7700 3000
@@
 Connection ~ 7700 2700
 $Comp
-L pcb-rescue:+3V3-power #PWR0203
+L pcb-rescue:+3V3-power-pcb-rescue #PWR0203
 U 1 1 5D1E3230
 P 8100 1800
@@
 $EndComp
 $Comp
-L pcb-rescue:IRLML6402-Transistor_FET Q300
+L pcb-rescue:IRLML6402-Transistor_FET-pcb-rescue Q300
 U 1 1 5D1E5978
 P 8000 2100
@@
 	7150 5100 8400 5100
 $Comp
-L pcb-rescue:R-Device R305
+L pcb-rescue:R-Device-pcb-rescue R305
 U 1 1 5D1FE40C
 P 7600 2350
@@
 $EndComp
 $Comp
-L pcb-rescue:R-Device R304
+L pcb-rescue:R-Device-pcb-rescue R304
 U 1 1 5D1FF47A
 P 7600 1850
@@
 	7600 2200 7600 2100
 $Comp
-L pcb-rescue:GND-power #PWR0204
+L pcb-rescue:GND-power-pcb-rescue #PWR0204
 U 1 1 5D20AD53
 P 7600 2500
@@
 $EndComp
 $Comp
-L pcb-rescue:+3V3-power #PWR0205
+L pcb-rescue:+3V3-power-pcb-rescue #PWR0205
 U 1 1 5D20B20B
 P 7600 1700
@@
 $EndComp
 $Comp
-L pcb-rescue:D_Schottky-Device D300
+L pcb-rescue:D_Schottky-Device-pcb-rescue D300
 U 1 1 5D20C1D1
 P 7350 2100
@@
 	7150 5200 7150 5100
 $Comp
-L pcb-rescue:GND-power #PWR0206
+L pcb-rescue:GND-power-pcb-rescue #PWR0206
 U 1 1 5D24A79B
 P 8400 6200
@@
 	8400 6100 8400 6200
 $Comp
-L pcb-rescue:C-Device C303
+L pcb-rescue:C-Device-pcb-rescue C303
 U 1 1 5D24DBD3
 P 8800 5250
@@
 $EndComp
 $Comp
-L pcb-rescue:C-Device C304
+L pcb-rescue:C-Device-pcb-rescue C304
 U 1 1 5D24DBD9
 P 9200 5250
@@
 $EndComp
 $Comp
-L pcb-rescue:GND-power #PWR0207
+L pcb-rescue:GND-power-pcb-rescue #PWR0207
 U 1 1 5D24DBDF
 P 8800 5400
@@
 	7500 2100 7600 2100
 $Comp
-L pcb-rescue:C-Device C305
+L pcb-rescue:C-Device-pcb-rescue C305
 U 1 1 5D259DFD
 P 2600 7250
@@
 	2600 7000 2600 7100
 $Comp
-L pcb-rescue:GND-power #PWR0208
+L pcb-rescue:GND-power-pcb-rescue #PWR0208
 U 1 1 5D25D3D4
 P 2600 7400
@@
 $EndComp
 $Comp
-L pcb-rescue:C-Device C306
+L pcb-rescue:C-Device-pcb-rescue C306
 U 1 1 5D25F58F
 P 2600 2650
@@
 $EndComp
 $Comp
-L pcb-rescue:GND-power #PWR0209
+L pcb-rescue:GND-power-pcb-rescue #PWR0209
 U 1 1 5D2600DE
 P 2600 2900
@@
 	2600 2900 2600 2800
 $Comp
-L pcb-rescue:+3V3-power #PWR0210
+L pcb-rescue:+3V3-power-pcb-rescue #PWR0210
 U 1 1 5D2689FB
 P 2600 4900
@@
 $EndComp
 $Comp
-L pcb-rescue:C-Device C308
+L pcb-rescue:C-Device-pcb-rescue C308
 U 1 1 5D268A01
 P 2600 5250
@@
 $EndComp
 $Comp
-L pcb-rescue:GND-power #PWR0211
+L pcb-rescue:GND-power-pcb-rescue #PWR0211
 U 1 1 5D268A07
 P 2600 5500
@@
 	2600 5500 2600 5400
 $Comp
-L pcb-rescue:+3V3-power #PWR0212
+L pcb-rescue:+3V3-power-pcb-rescue #PWR0212
 U 1 1 5D26D067
 P 2600 5900
@@
 $EndComp
 $Comp
-L pcb-rescue:C-Device C309
+L pcb-rescue:C-Device-pcb-rescue C309
 U 1 1 5D26D06D
 P 2600 6250
@@
 $EndComp
 $Comp
-L pcb-rescue:GND-power #PWR0213
+L pcb-rescue:GND-power-pcb-rescue #PWR0213
 U 1 1 5D26D073
 P 2600 6500
@@
 Connection ~ 2600 5900
 $Comp
-L pcb-rescue:C-Device C307
+L pcb-rescue:C-Device-pcb-rescue C307
 U 1 1 5D273248
 P 2600 4250
@@
 $EndComp
 $Comp
-L pcb-rescue:GND-power #PWR0214
+L pcb-rescue:GND-power-pcb-rescue #PWR0214
 U 1 1 5D27324E
 P 2600 4500
@@
 	2600 4500 2600 4400
 $Comp
-L pcb-rescue:ADP7142AUZJ-Regulator_Linear U300
+L pcb-rescue:ADP7142AUZJ-Regulator_Linear-pcb-rescue U300
 U 1 1 5D27B732
 P 3800 1000
@@
 Connection ~ 6400 4100
 $Comp
-L pcb-rescue:GND-power #PWR0215
+L pcb-rescue:GND-power-pcb-rescue #PWR0215
 U 1 1 5D39B0B3
 P 3800 1300
@@
 $EndComp
 $Comp
-L pcb-rescue:C-Device C310
+L pcb-rescue:C-Device-pcb-rescue C310
 U 1 1 5D39B62C
 P 2500 1050
@@
 $EndComp
 $Comp
-L pcb-rescue:C-Device C311
+L pcb-rescue:C-Device-pcb-rescue C311
 U 1 1 5D39C092
 P 2900 1050
@@
 $EndComp
 $Comp
-L pcb-rescue:Q_NMOS_SGD-Device Q302
+L pcb-rescue:Q_NMOS_SGD-Device-pcb-rescue Q302
 U 1 1 5D3A2E7B
 P 4900 1300
@@
 $EndComp
 $Comp
-L pcb-rescue:R-Device R307
+L pcb-rescue:R-Device-pcb-rescue R307
 U 1 1 5D3AB9EC
 P 4400 1350
@@
 $EndComp
 $Comp
-L pcb-rescue:R-Device R306
+L pcb-rescue:R-Device-pcb-rescue R306
 U 1 1 5D3ABE8A
 P 4400 1050
@@
 $EndComp
 $Comp
-L pcb-rescue:R-Device R308
+L pcb-rescue:R-Device-pcb-rescue R308
 U 1 1 5D3AF41C
 P 4900 1650
@@
 $EndComp
 $Comp
-L pcb-rescue:R-Device R309
+L pcb-rescue:R-Device-pcb-rescue R309
 U 1 1 5D3BF697
 P 5200 1050
@@
 $EndComp
 $Comp
-L pcb-rescue:C-Device C312
+L pcb-rescue:C-Device-pcb-rescue C312
 U 1 1 5D3C0823
 P 5600 1050
@@
 $EndComp
 $Comp
-L pcb-rescue:C-Device C313
+L pcb-rescue:C-Device-pcb-rescue C313
 U 1 1 5D3C0829
 P 6000 1050
@@
 $EndComp
 $Comp
-L pcb-rescue:GND-power #PWR0216
+L pcb-rescue:GND-power-pcb-rescue #PWR0216
 U 1 1 5D3C082F
 P 5600 1200
@@
 Connection ~ 5600 1200
 $Comp
-L pcb-rescue:GND-power #PWR0217
+L pcb-rescue:GND-power-pcb-rescue #PWR0217
 U 1 1 5D3CF6CC
 P 4900 1800
@@
 $EndComp
 $Comp
-L pcb-rescue:GND-power #PWR0218
+L pcb-rescue:GND-power-pcb-rescue #PWR0218
 U 1 1 5D3CFB51
 P 4400 1500
@@
 	2900 1200 2500 1200
 $Comp
-L pcb-rescue:GND-power #PWR0219
+L pcb-rescue:GND-power-pcb-rescue #PWR0219
 U 1 1 5D3FB2DA
 P 2500 1200
@@
 Connection ~ 2500 1200
 $Comp
-L pcb-rescue:+3V3-power #PWR0220
+L pcb-rescue:+3V3-power-pcb-rescue #PWR0220
 U 1 1 5D3FB6DC
 P 2500 900
@@
 FB = 0.5V, use 560K/487K/100K\nFB = 0.8V, use 499K/330K/160K\nFB = 1.0V, use 464K/243K/200K
 $Comp
-L pcb-rescue:+1V8-power #PWR0221
+L pcb-rescue:+1V8-power-pcb-rescue #PWR0221
 U 1 1 5D3F1E82
 P 8400 5000
@@
 Configure as 32kHz clock output
 $Comp
-L pcb-rescue:+1V8-power #PWR0222
+L pcb-rescue:+1V8-power-pcb-rescue #PWR0222
 U 1 1 5D2012F3
 P 2600 2300
