File: pcb/storage.sch (KiCad schematic (older format))
At the start: 31 parts, among them Q300 IRLML6402, Q302 2SK3018, U100 MCIMX7S5EVM08SC, U300 ADP123, U301 W25Q16BV

Commit message: pcb: remap schematic symbols
Parts:
- C300, C301, C302, C303, C304, C305, C306, C307, C308, C309, C310, C311, C312, C313: symbol pcb-rescue:C-Device-pcb-rescue -> Device:C
- D300: symbol pcb-rescue:D_Schottky-Device-pcb-rescue -> Device:D_Schottky
- Q300: symbol pcb-rescue:IRLML6402-Transistor_FET-pcb-rescue -> Transistor_FET:IRLML6402
- Q302: symbol pcb-rescue:Q_NMOS_SGD-Device-pcb-rescue -> Device:Q_NMOS_SGD
- R300, R301, R302, R303, R304, R305, R306, R307, R308, R309: symbol pcb-rescue:R-Device-pcb-rescue -> Device:R
- U300: symbol pcb-rescue:ADP7142AUZJ-Regulator_Linear-pcb-rescue -> Regulator_Linear:ADP7142AUJZ
Connections:
- net at Q302.1 (S), R306.2, R307.1: no longer U300.4 (FB)
Changed lines of the file:
@@
 	6900 3700 7400 3700
 $Comp
-L pcb-rescue:GND-power-pcb-rescue #PWR0200
+L power:GND #PWR0200
 U 1 1 5DBA2B48
 P 7300 4300
@@
 To Audio DAC\n
 $Comp
-L pcb-rescue:R-Device-pcb-rescue R300
+L Device:R R300
 U 1 1 5DBBE698
 P 7150 5350
@@
 $EndComp
 $Comp
-L pcb-rescue:R-Device-pcb-rescue R301
+L Device:R R301
 U 1 1 5DBC08BA
 P 6400 2950
@@
 $EndComp
 $Comp
-L pcb-rescue:R-Device-pcb-rescue R302
+L Device:R R302
 U 1 1 5DBC0C88
 P 5900 2950
@@
 $EndComp
 $Comp
-L pcb-rescue:R-Device-pcb-rescue R303
+L Device:R R303
 U 1 1 5DBC2BE9
 P 6650 3700
@@
 	5900 2800 5900 2700
 $Comp
-L pcb-rescue:C-Device-pcb-rescue C300
+L Device:C C300
 U 1 1 5DBD27EC
 P 6900 4350
@@
 $EndComp
 $Comp
-L pcb-rescue:GND-power-pcb-rescue #PWR0201
+L power:GND #PWR0201
 U 1 1 5DBD7168
 P 6900 4600
@@
 	6900 4500 6900 4600
 $Comp
-L pcb-rescue:C-Device-pcb-rescue C301
+L Device:C C301
 U 1 1 5DBD9F72
 P 7700 2850
@@
 $EndComp
 $Comp
-L pcb-rescue:C-Device-pcb-rescue C302
+L Device:C C302
 U 1 1 5DBDAEE7
 P 8100 2850
@@
 $EndComp
 $Comp
-L pcb-rescue:GND-power-pcb-rescue #PWR0202
+L power:GND #PWR0202
 U 1 1 5DBDB16E
 P 7700 3000
@@
 Connection ~ 7700 2700
 $Comp
-L pcb-rescue:+3V3-power-pcb-rescue #PWR0203
+L power:+3V3 #PWR0203
 U 1 1 5D1E3230
 P 8100 1800
@@
 $EndComp
 $Comp
-L pcb-rescue:IRLML6402-Transistor_FET-pcb-rescue Q300
+L Transistor_FET:IRLML6402 Q300
 U 1 1 5D1E5978
 P 8000 2100
@@
 	7150 5100 8400 5100
 $Comp
-L pcb-rescue:R-Device-pcb-rescue R305
+L Device:R R305
 U 1 1 5D1FE40C
 P 7600 2350
@@
 $EndComp
 $Comp
-L pcb-rescue:R-Device-pcb-rescue R304
+L Device:R R304
 U 1 1 5D1FF47A
 P 7600 1850
@@
 	7600 2200 7600 2100
 $Comp
-L pcb-rescue:GND-power-pcb-rescue #PWR0204
+L power:GND #PWR0204
 U 1 1 5D20AD53
 P 7600 2500
@@
 $EndComp
 $Comp
-L pcb-rescue:+3V3-power-pcb-rescue #PWR0205
+L power:+3V3 #PWR0205
 U 1 1 5D20B20B
 P 7600 1700
@@
 $EndComp
 $Comp
-L pcb-rescue:D_Schottky-Device-pcb-rescue D300
+L Device:D_Schottky D300
 U 1 1 5D20C1D1
 P 7350 2100
@@
 	7150 5200 7150 5100
 $Comp
-L pcb-rescue:GND-power-pcb-rescue #PWR0206
+L power:GND #PWR0206
 U 1 1 5D24A79B
 P 8400 6200
@@
 	8400 6100 8400 6200
 $Comp
-L pcb-rescue:C-Device-pcb-rescue C303
+L Device:C C303
 U 1 1 5D24DBD3
 P 8800 5250
@@
 $EndComp
 $Comp
-L pcb-rescue:C-Device-pcb-rescue C304
+L Device:C C304
 U 1 1 5D24DBD9
 P 9200 5250
@@
 $EndComp
 $Comp
-L pcb-rescue:GND-power-pcb-rescue #PWR0207
+L power:GND #PWR0207
 U 1 1 5D24DBDF
 P 8800 5400
@@
 	7500 2100 7600 2100
 $Comp
-L pcb-rescue:C-Device-pcb-rescue C305
+L Device:C C305
 U 1 1 5D259DFD
 P 2600 7250
@@
 	2600 7000 2600 7100
 $Comp
-L pcb-rescue:GND-power-pcb-rescue #PWR0208
+L power:GND #PWR0208
 U 1 1 5D25D3D4
 P 2600 7400
@@
 $EndComp
 $Comp
-L pcb-rescue:C-Device-pcb-rescue C306
+L Device:C C306
 U 1 1 5D25F58F
 P 2600 2650
@@
 $EndComp
 $Comp
-L pcb-rescue:GND-power-pcb-rescue #PWR0209
+L power:GND #PWR0209
 U 1 1 5D2600DE
 P 2600 2900
@@
 	2600 2900 2600 2800
 $Comp
-L pcb-rescue:+3V3-power-pcb-rescue #PWR0210
+L power:+3V3 #PWR0210
 U 1 1 5D2689FB
 P 2600 4900
@@
 $EndComp
 $Comp
-L pcb-rescue:C-Device-pcb-rescue C308
+L Device:C C308
 U 1 1 5D268A01
 P 2600 5250
@@
 $EndComp
 $Comp
-L pcb-rescue:GND-power-pcb-rescue #PWR0211
+L power:GND #PWR0211
 U 1 1 5D268A07
 P 2600 5500
@@
 	2600 5500 2600 5400
 $Comp
-L pcb-rescue:+3V3-power-pcb-rescue #PWR0212
+L power:+3V3 #PWR0212
 U 1 1 5D26D067
 P 2600 5900
@@
 $EndComp
 $Comp
-L pcb-rescue:C-Device-pcb-rescue C309
+L Device:C C309
 U 1 1 5D26D06D
 P 2600 6250
@@
 $EndComp
 $Comp
-L pcb-rescue:GND-power-pcb-rescue #PWR0213
+L power:GND #PWR0213
 U 1 1 5D26D073
 P 2600 6500
@@
 Connection ~ 2600 5900
 $Comp
-L pcb-rescue:C-Device-pcb-rescue C307
+L Device:C C307
 U 1 1 5D273248
 P 2600 4250
@@
 $EndComp
 $Comp
-L pcb-rescue:GND-power-pcb-rescue #PWR0214
+L power:GND #PWR0214
 U 1 1 5D27324E
 P 2600 4500
@@
 	2600 4500 2600 4400
 $Comp
-L pcb-rescue:ADP7142AUZJ-Regulator_Linear-pcb-rescue U300
+L Regulator_Linear:ADP7142AUJZ U300
 U 1 1 5D27B732
 P 3800 1000
@@
 Connection ~ 6400 4100
 $Comp
-L pcb-rescue:GND-power-pcb-rescue #PWR0215
+L power:GND #PWR0215
 U 1 1 5D39B0B3
 P 3800 1300
@@
 $EndComp
 $Comp
-L pcb-rescue:C-Device-pcb-rescue C310
+L Device:C C310
 U 1 1 5D39B62C
 P 2500 1050
@@
 $EndComp
 $Comp
-L pcb-rescue:C-Device-pcb-rescue C311
+L Device:C C311
 U 1 1 5D39C092
 P 2900 1050
@@
 $EndComp
 $Comp
-L pcb-rescue:Q_NMOS_SGD-Device-pcb-rescue Q302
+L Device:Q_NMOS_SGD Q302
 U 1 1 5D3A2E7B
 P 4900 1300
@@
 $EndComp
 $Comp
-L pcb-rescue:R-Device-pcb-rescue R307
+L Device:R R307
 U 1 1 5D3AB9EC
 P 4400 1350
@@
 $EndComp
 $Comp
-L pcb-rescue:R-Device-pcb-rescue R306
+L Device:R R306
 U 1 1 5D3ABE8A
 P 4400 1050
@@
 $EndComp
 $Comp
-L pcb-rescue:R-Device-pcb-rescue R308
+L Device:R R308
 U 1 1 5D3AF41C
 P 4900 1650
@@
 $EndComp
 $Comp
-L pcb-rescue:R-Device-pcb-rescue R309
+L Device:R R309
 U 1 1 5D3BF697
 P 5200 1050
@@
 $EndComp
 $Comp
-L pcb-rescue:C-Device-pcb-rescue C312
+L Device:C C312
 U 1 1 5D3C0823
 P 5600 1050
@@
 $EndComp
 $Comp
-L pcb-rescue:C-Device-pcb-rescue C313
+L Device:C C313
 U 1 1 5D3C0829
 P 6000 1050
@@
 $EndComp
 $Comp
-L pcb-rescue:GND-power-pcb-rescue #PWR0216
+L power:GND #PWR0216
 U 1 1 5D3C082F
 P 5600 1200
@@
 Connection ~ 5600 1200
 $Comp
-L pcb-rescue:GND-power-pcb-rescue #PWR0217
+L power:GND #PWR0217
 U 1 1 5D3CF6CC
 P 4900 1800
@@
 $EndComp
 $Comp
-L pcb-rescue:GND-power-pcb-rescue #PWR0218
+L power:GND #PWR0218
 U 1 1 5D3CFB51
 P 4400 1500
@@
 	2900 1200 2500 1200
 $Comp
-L pcb-rescue:GND-power-pcb-rescue #PWR0219
+L power:GND #PWR0219
 U 1 1 5D3FB2DA
 P 2500 1200
@@
 Connection ~ 2500 1200
 $Comp
-L pcb-rescue:+3V3-power-pcb-rescue #PWR0220
+L power:+3V3 #PWR0220
 U 1 1 5D3FB6DC
 P 2500 900
@@
 FB = 0.5V, use 560K/487K/100K\nFB = 0.8V, use 499K/330K/160K\nFB = 1.0V, use 464K/243K/200K
 $Comp
-L pcb-rescue:+1V8-power-pcb-rescue #PWR0221
+L power:+1V8 #PWR0221
 U 1 1 5D3F1E82
 P 8400 5000
@@
 Configure as 32kHz clock output
 $Comp
-L pcb-rescue:+1V8-power-pcb-rescue #PWR0222
+L power:+1V8 #PWR0222
 U 1 1 5D2012F3
 P 2600 2300

Commit message: fix #2
Connections:
- net at U300.4 (SENSE/ADJ): now also Q302.1 (S), R306.2, R307.1
Changed lines of the file:
@@
 Connection ~ 4400 1200
-Wire Wire Line
-	4200 1100 4200 1200
 Wire Wire Line
 	4200 1200 4400 1200
@@
 NoConn ~ 4400 3600
 NoConn ~ 4400 3700
+Wire Wire Line
+	4200 1000 4200 1200
 $EndSCHEMATC
