File: pcb/unused.sch (KiCad schematic (older format))
At the start: 0 parts

Commit message: pcb: working on sch
Parts:
- added U100: MCIMX7S5EVM08SC, footprints:BGA-541_25x25_19.0x19.0mm, symbol symbols:MCIMX7S5EVM08SC
Changed lines of the file:
@@
 $Descr A4 11693 8268
 encoding utf-8
-Sheet 1 11
+Sheet 9 11
 Title ""
 Date ""
@@
 Comment4 ""
 $EndDescr
+$Comp
+L symbols:MCIMX7S5EVM08SC U100
+U 5 1 5D617663
+P 2700 4700
+F 0 "U100" H 2700 7065 50  0000 C CNN
+F 1 "MCIMX7S5EVM08SC" H 2700 6974 50  0000 C CNN
+F 2 "footprints:BGA-541_25x25_19.0x19.0mm" H 2700 5400 50  0001 C CNN
+F 3 "" H 2700 5400 50  0001 C CNN
+	5    2700 4700
+	1    0    0    -1
+$EndComp
+$Comp
+L symbols:MCIMX7S5EVM08SC U100
+U 11 1 5D62E3CD
+P 5800 5100
+F 0 "U100" H 5858 7465 50  0000 C CNN
+F 1 "MCIMX7S5EVM08SC" H 5858 7374 50  0000 C CNN
+F 2 "footprints:BGA-541_25x25_19.0x19.0mm" H 5800 5800 50  0001 C CNN
+F 3 "" H 5800 5800 50  0001 C CNN
+	11   5800 5100
+	1    0    0    -1
+$EndComp
+$Comp
+L symbols:MCIMX7S5EVM08SC U100
+U 12 1 5D643A6C
+P 8900 4800
+F 0 "U100" H 8958 7165 50  0000 C CNN
+F 1 "MCIMX7S5EVM08SC" H 8958 7074 50  0000 C CNN
+F 2 "footprints:BGA-541_25x25_19.0x19.0mm" H 8900 5500 50  0001 C CNN
+F 3 "" H 8900 5500 50  0001 C CNN
+	12   8900 4800
+	1    0    0    -1
+$EndComp
 $EndSCHEMATC

Commit message: pcb: working on sch
Connections:
- net GND: now reaches U100.H16 (NVCC_ENET1)
- net GND: now also U100.AA13 (PCIE_REXT)
- no-connect marks 0 -> 37
Changed lines of the file:
@@
 	1    0    0    -1
 $EndComp
+$Comp
+L power:GND #PWR?
+U 1 1 5D1F6AB8
+P 6700 4400
+F 0 "#PWR?" H 6700 4150 50  0001 C CNN
+F 1 "GND" H 6705 4227 50  0000 C CNN
+F 2 "" H 6700 4400 50  0001 C CNN
+F 3 "" H 6700 4400 50  0001 C CNN
+	1    6700 4400
+	1    0    0    -1
+$EndComp
+Wire Wire Line
+	6600 4300 6700 4300
+Wire Wire Line
+	6700 4300 6700 4400
+NoConn ~ 6600 3100
+NoConn ~ 6600 3200
+NoConn ~ 6600 3400
+NoConn ~ 6600 3500
+NoConn ~ 6600 3700
+NoConn ~ 6600 3800
+NoConn ~ 6600 4000
+NoConn ~ 6600 4100
+NoConn ~ 9700 2800
+NoConn ~ 9700 2900
+NoConn ~ 9700 3100
+NoConn ~ 9700 3200
+NoConn ~ 9700 3400
+NoConn ~ 9700 3500
+NoConn ~ 9700 3700
+NoConn ~ 9700 3800
+NoConn ~ 9700 4000
+NoConn ~ 9700 4100
+NoConn ~ 9700 4300
+NoConn ~ 9700 4400
+NoConn ~ 3500 2700
+NoConn ~ 3500 2800
+NoConn ~ 3500 2900
+NoConn ~ 3500 3000
+NoConn ~ 3500 3200
+NoConn ~ 3500 3300
+NoConn ~ 3500 3400
+NoConn ~ 3500 3600
+NoConn ~ 3500 3700
+NoConn ~ 3500 3800
+NoConn ~ 3500 3900
+NoConn ~ 3500 4100
+NoConn ~ 3500 4200
+NoConn ~ 3500 4300
+NoConn ~ 3500 4500
+NoConn ~ 3500 4600
+NoConn ~ 1900 4500
+$Comp
+L power:GND #PWR?
+U 1 1 5D208234
+P 1800 2800
+F 0 "#PWR?" H 1800 2550 50  0001 C CNN
+F 1 "GND" H 1805 2627 50  0000 C CNN
+F 2 "" H 1800 2800 50  0001 C CNN
+F 3 "" H 1800 2800 50  0001 C CNN
+	1    1800 2800
+	1    0    0    -1
+$EndComp
+Wire Wire Line
+	1900 2700 1800 2700
+Wire Wire Line
+	1800 2700 1800 2800
 $EndSCHEMATC
