File: pcb/wifibt.sch (KiCad schematic (older format))
At the start: 15 parts, among them Q800 IRLML6402, U800 RTL8723BS

Commit message: pcb: remap schematic symbols
Parts:
- C800, C801, C802, C803, C804, C805, C806: symbol pcb-rescue:C-Device-pcb-rescue -> Device:C
- D800: symbol pcb-rescue:D_Schottky-Device-pcb-rescue -> Device:D_Schottky
- Q800: symbol pcb-rescue:IRLML6402-Transistor_FET-pcb-rescue -> Transistor_FET:IRLML6402
- R800, R801, R802, R803: symbol pcb-rescue:R-Device-pcb-rescue -> Device:R
Changed lines of the file:
@@
 $EndComp
 $Comp
-L pcb-rescue:C-Device-pcb-rescue C800
+L Device:C C800
 U 1 1 5D1C38FE
 P 6700 3450
@@
 $EndComp
 $Comp
-L pcb-rescue:C-Device-pcb-rescue C801
+L Device:C C801
 U 1 1 5D1C53ED
 P 7200 3450
@@
 $EndComp
 $Comp
-L pcb-rescue:C-Device-pcb-rescue C802
+L Device:C C802
 U 1 1 5D1C595A
 P 7700 3450
@@
 $EndComp
 $Comp
-L pcb-rescue:C-Device-pcb-rescue C803
+L Device:C C803
 U 1 1 5D1C5D04
 P 8200 3450
@@
 $EndComp
 $Comp
-L pcb-rescue:GND-power-pcb-rescue #PWR0306
+L power:GND #PWR0306
 U 1 1 5D1C6F63
 P 7700 3700
@@
 $EndComp
 $Comp
-L pcb-rescue:+3V3-power-pcb-rescue #PWR?
+L power:+3V3 #PWR?
 U 1 1 5D1E0260
 P 6700 1900
@@
 $EndComp
 $Comp
-L pcb-rescue:IRLML6402-Transistor_FET-pcb-rescue Q?
+L Transistor_FET:IRLML6402 Q?
 U 1 1 5D1E0266
 P 6600 2200
@@
 	6700 1900 6700 2000
 $Comp
-L pcb-rescue:R-Device-pcb-rescue R?
+L Device:R R?
 U 1 1 5D1E026D
 P 6200 2450
@@
 $EndComp
 $Comp
-L pcb-rescue:R-Device-pcb-rescue R?
+L Device:R R?
 U 1 1 5D1E0273
 P 6200 1950
@@
 	6200 2300 6200 2200
 $Comp
-L pcb-rescue:GND-power-pcb-rescue #PWR?
+L power:GND #PWR?
 U 1 1 5D1E027E
 P 6200 2600
@@
 $EndComp
 $Comp
-L pcb-rescue:+3V3-power-pcb-rescue #PWR?
+L power:+3V3 #PWR?
 U 1 1 5D1E0284
 P 6200 1800
@@
 $EndComp
 $Comp
-L pcb-rescue:D_Schottky-Device-pcb-rescue D?
+L Device:D_Schottky D?
 U 1 1 5D1E028A
 P 5950 2200
@@
 Connection ~ 7700 3600
 $Comp
-L pcb-rescue:GND-power-pcb-rescue #PWR0310
+L power:GND #PWR0310
 U 1 1 5D1C677C
 P 6700 3700
@@
 $EndComp
 $Comp
-L pcb-rescue:GND-power-pcb-rescue #PWR0311
+L power:GND #PWR0311
 U 1 1 5D1E38E1
 P 6500 3900
@@
 	6500 3500 6500 3600
 $Comp
-L pcb-rescue:C-Device-pcb-rescue C804
+L Device:C C804
 U 1 1 5D1E5233
 P 4850 5400
@@
 $EndComp
 $Comp
-L pcb-rescue:C-Device-pcb-rescue C805
+L Device:C C805
 U 1 1 5D1E5893
 P 4600 5650
@@
 $EndComp
 $Comp
-L pcb-rescue:R-Device-pcb-rescue R?
+L Device:R R?
 U 1 1 5D1E5CB8
 P 4350 5400
@@
 $EndComp
 $Comp
-L pcb-rescue:C-Device-pcb-rescue C806
+L Device:C C806
 U 1 1 5D1E62F9
 P 4100 5650
@@
 $EndComp
 $Comp
-L pcb-rescue:GND-power-pcb-rescue #PWR0312
+L power:GND #PWR0312
 U 1 1 5D1EA804
 P 3700 5600
@@
 $EndComp
 $Comp
-L pcb-rescue:GND-power-pcb-rescue #PWR0313
+L power:GND #PWR0313
 U 1 1 5D1EAE49
 P 4100 5900
@@
 $EndComp
 $Comp
-L pcb-rescue:GND-power-pcb-rescue #PWR0314
+L power:GND #PWR0314
 U 1 1 5D1EB029
 P 4600 5900
@@
 $EndComp
 $Comp
-L pcb-rescue:GND-power-pcb-rescue #PWR0315
+L power:GND #PWR0315
 U 1 1 5D1EB239
 P 5100 5600
@@
 	4700 3800 5200 3800
 $Comp
-L pcb-rescue:R-Device-pcb-rescue R?
+L Device:R R?
 U 1 1 5D20325E
 P 5100 2850
