File: pcb/audio.sch (KiCad schematic (older format))
At the start: 32 parts, among them J1 AudioJack3_SwitchTR, U400 CS43130, U401 ADP150-3.0, U402 ADP150-1.8, U403 ADP150-1.8, X400 DSC1001CE2-022.5792

Commit message: pcb: remap schematic symbols
Parts:
- C400, C401, C402, C403, C404, C405, C406, C407, C408, C409, C410, C411, C412, C413, C414, C415, C416, C417: symbol pcb-rescue:C-Device-pcb-rescue -> Device:C
- J1: symbol pcb-rescue:AudioJack3_SwitchTR-Connector-pcb-rescue -> Connector:AudioJack3_SwitchTR
- L400, L401: symbol pcb-rescue:L-Device-pcb-rescue -> Device:L_Small
- R400, R401, R402, R403, R404: symbol pcb-rescue:R-Device-pcb-rescue -> Device:R
- RV400: symbol pcb-rescue:R_POT-Device-pcb-rescue -> Device:R_POT
- U401: symbol pcb-rescue:AP2127K-3.0-Regulator_Linear-pcb-rescue -> Regulator_Linear:AP2127K-3.0
- U402, U403: symbol pcb-rescue:AP2112K-1.8-Regulator_Linear-pcb-rescue -> Regulator_Linear:AP2112K-1.8
- X400: symbol pcb-rescue:ASE-xxxMHz-Oscillator-pcb-rescue -> Oscillator:ASE-xxxMHz
Connections:
- net +1V8: no longer L400.1, L401.1
- net at C401.1, C402.1, U400.31 (VL)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: no longer L401.2
- net at C400.1, X400.1 (EN), X400.4 (Vdd): no longer L400.2
Changed lines of the file:
@@
 $EndComp
 $Comp
-L pcb-rescue:AP2112K-1.8-Regulator_Linear-pcb-rescue U402
+L Regulator_Linear:AP2112K-1.8 U402
 U 1 1 5D3BE239
 P 8200 3500
@@
 $EndComp
 $Comp
-L pcb-rescue:AP2127K-3.0-Regulator_Linear-pcb-rescue U401
+L Regulator_Linear:AP2127K-3.0 U401
 U 1 1 5D3C4251
 P 8200 2500
@@
 $EndComp
 $Comp
-L pcb-rescue:+3V3-power-pcb-rescue #PWR0252
+L power:+3V3 #PWR0252
 U 1 1 5D3C5E19
 P 8600 2300
@@
 	8500 2500 8600 2500
 $Comp
-L pcb-rescue:GND-power-pcb-rescue #PWR0253
+L power:GND #PWR0253
 U 1 1 5D3C6CEC
 P 8200 2800
@@
 $EndComp
 $Comp
-L pcb-rescue:GND-power-pcb-rescue #PWR0254
+L power:GND #PWR0254
 U 1 1 5D3C71EE
 P 8200 3800
@@
 $EndComp
 $Comp
-L pcb-rescue:C-Device-pcb-rescue C405
+L Device:C C405
 U 1 1 5D3C76A9
 P 8900 2550
@@
 $EndComp
 $Comp
-L pcb-rescue:C-Device-pcb-rescue C408
+L Device:C C408
 U 1 1 5D3C8004
 P 8900 3550
@@
 $EndComp
 $Comp
-L pcb-rescue:C-Device-pcb-rescue C404
+L Device:C C404
 U 1 1 5D3C85BE
 P 7600 2550
@@
 $EndComp
 $Comp
-L pcb-rescue:C-Device-pcb-rescue C407
+L Device:C C407
 U 1 1 5D3C8D9A
 P 7700 3550
@@
 $EndComp
 $Comp
-L pcb-rescue:C-Device-pcb-rescue C406
+L Device:C C406
 U 1 1 5D3C9210
 P 7300 3650
@@
 $EndComp
 $Comp
-L pcb-rescue:C-Device-pcb-rescue C403
+L Device:C C403
 U 1 1 5D3C9FD4
 P 7200 2550
@@
 $EndComp
 $Comp
-L pcb-rescue:GND-power-pcb-rescue #PWR0255
+L power:GND #PWR0255
 U 1 1 5D3CA6E5
 P 7600 2700
@@
 $EndComp
 $Comp
-L pcb-rescue:GND-power-pcb-rescue #PWR0256
+L power:GND #PWR0256
 U 1 1 5D3CA8EB
 P 7200 2700
@@
 $EndComp
 $Comp
-L pcb-rescue:GND-power-pcb-rescue #PWR0257
+L power:GND #PWR0257
 U 1 1 5D3CAA8D
 P 8900 2700
@@
 $EndComp
 $Comp
-L pcb-rescue:GND-power-pcb-rescue #PWR0258
+L power:GND #PWR0258
 U 1 1 5D3CAE2F
 P 8900 3700
@@
 $EndComp
 $Comp
-L pcb-rescue:GND-power-pcb-rescue #PWR0259
+L power:GND #PWR0259
 U 1 1 5D3CB31E
 P 7700 3700
@@
 $EndComp
 $Comp
-L pcb-rescue:GND-power-pcb-rescue #PWR0260
+L power:GND #PWR0260
 U 1 1 5D3CB6C2
 P 7300 3800
@@
 Connection ~ 8600 2500
 $Comp
-L pcb-rescue:C-Device-pcb-rescue C410
+L Device:C C410
 U 1 1 5D3CDB2E
 P 6950 3300
@@
 $EndComp
 $Comp
-L pcb-rescue:C-Device-pcb-rescue C411
+L Device:C C411
 U 1 1 5D3CEBF2
 P 6950 3600
@@
 $EndComp
 $Comp
-L pcb-rescue:C-Device-pcb-rescue C412
+L Device:C C412
 U 1 1 5D3D16A3
 P 6950 3800
@@
 	6800 3800 6600 3800
 $Comp
-L pcb-rescue:AP2112K-1.8-Regulator_Linear-pcb-rescue U403
+L Regulator_Linear:AP2112K-1.8 U403
 U 1 1 5D3DDAF9
 P 8200 4400
@@
 Connection ~ 8600 4300
 $Comp
-L pcb-rescue:GND-power-pcb-rescue #PWR0261
+L power:GND #PWR0261
 U 1 1 5D3DDB03
 P 8200 4700
@@
 $EndComp
 $Comp
-L pcb-rescue:C-Device-pcb-rescue C409
+L Device:C C409
 U 1 1 5D3DDB09
 P 8900 4450
@@
 $EndComp
 $Comp
-L pcb-rescue:C-Device-pcb-rescue C417
+L Device:C C417
 U 1 1 5D3DDB0F
 P 7700 4450
@@
 $EndComp
 $Comp
-L pcb-rescue:GND-power-pcb-rescue #PWR0262
+L power:GND #PWR0262
 U 1 1 5D3DDB15
 P 8900 4600
@@
 $EndComp
 $Comp
-L pcb-rescue:GND-power-pcb-rescue #PWR0263
+L power:GND #PWR0263
 U 1 1 5D3DDB1B
 P 7700 4600
@@
 Connection ~ 7700 4300
 $Comp
-L pcb-rescue:C-Device-pcb-rescue C416
+L Device:C C416
 U 1 1 5D3E2D8A
 P 7400 4350
@@
 $EndComp
 $Comp
-L pcb-rescue:C-Device-pcb-rescue C415
+L Device:C C415
 U 1 1 5D3E3537
 P 7100 4450
@@
 $EndComp
 $Comp
-L pcb-rescue:C-Device-pcb-rescue C413
+L Device:C C413
 U 1 1 5D3E42FA
 P 6750 4500
@@
 $EndComp
 $Comp
-L pcb-rescue:C-Device-pcb-rescue C414
+L Device:C C414
 U 1 1 5D3E4B00
 P 6750 4700
@@
 $EndComp
 $Comp
-L pcb-rescue:GND-power-pcb-rescue #PWR0264
+L power:GND #PWR0264
 U 1 1 5D3E50F6
 P 7400 4500
@@
 $EndComp
 $Comp
-L pcb-rescue:GND-power-pcb-rescue #PWR0265
+L power:GND #PWR0265
 U 1 1 5D3E5385
 P 7100 4600
@@
 $EndComp
 $Comp
-L pcb-rescue:GND-power-pcb-rescue #PWR0266
+L power:GND #PWR0266
 U 1 1 5D3E55AD
 P 6600 4400
@@
 	7150 5200 6600 5200
 $Comp
-L pcb-rescue:+1V8-power-pcb-rescue #PWR0267
+L power:+1V8 #PWR0267
 U 1 1 5D40EC46
 P 4200 2300
@@
 $EndComp
 $Comp
-L pcb-rescue:C-Device-pcb-rescue C402
+L Device:C C402
 U 1 1 5D412186
 P 4600 2750
@@
 $EndComp
 $Comp
-L pcb-rescue:GND-power-pcb-rescue #PWR0268
+L power:GND #PWR0268
 U 1 1 5D41218C
 P 4600 2900
@@
 $EndComp
 $Comp
-L pcb-rescue:C-Device-pcb-rescue C401
+L Device:C C401
 U 1 1 5D414243
 P 4200 2750
@@
 $EndComp
 $Comp
-L pcb-rescue:GND-power-pcb-rescue #PWR0269
+L power:GND #PWR0269
 U 1 1 5D414249
 P 4200 2900
@@
 SAI1_MCLK
 $Comp
-L pcb-rescue:R-Device-pcb-rescue R400
+L Device:R R400
 U 1 1 5D42CABC
 P 4650 3300
@@
 $EndComp
 $Comp
-L pcb-rescue:R-Device-pcb-rescue R401
+L Device:R R401
 U 1 1 5D437A63
 P 4650 4100
@@
 $EndComp
 $Comp
-L pcb-rescue:R-Device-pcb-rescue R402
+L Device:R R402
 U 1 1 5D438FF1
 P 4650 4200
@@
 $EndComp
 $Comp
-L pcb-rescue:R-Device-pcb-rescue R403
+L Device:R R403
 U 1 1 5D4391CB
 P 4650 4300
@@
 	4800 4300 5000 4300
 $Comp
-L pcb-rescue:GND-power-pcb-rescue #PWR0270
+L power:GND #PWR0270
 U 1 1 5D44FB8A
 P 4900 5700
@@
 	4300 5200 5000 5200
 $Comp
-L pcb-rescue:R-Device-pcb-rescue R404
+L Device:R R404
 U 1 1 5D46D440
 P 4650 5300
@@
 $EndComp
 $Comp
-L pcb-rescue:+1V8-power-pcb-rescue #PWR0271
+L power:+1V8 #PWR0271
 U 1 1 5D46FEBD
 P 4300 5300
@@
 NoConn ~ 5000 3600
 $Comp
-L pcb-rescue:ASE-xxxMHz-Oscillator-pcb-rescue X400
+L Oscillator:ASE-xxxMHz X400
 U 1 1 5D484130
 P 3500 3500
@@
 $EndComp
 $Comp
-L pcb-rescue:+1V8-power-pcb-rescue #PWR0272
+L power:+1V8 #PWR0272
 U 1 1 5D485FE4
 P 3500 2300
@@
 $EndComp
 $Comp
-L pcb-rescue:C-Device-pcb-rescue C400
+L Device:C C400
 U 1 1 5D487832
 P 3100 2750
@@
 $EndComp
 $Comp
-L pcb-rescue:GND-power-pcb-rescue #PWR0273
+L power:GND #PWR0273
 U 1 1 5D487838
 P 3100 2900
@@
 Connection ~ 3500 2600
 $Comp
-L pcb-rescue:GND-power-pcb-rescue #PWR0274
+L power:GND #PWR0274
 U 1 1 5D490333
 P 3500 3800
@@
 	3800 3500 5000 3500
 $Comp
-L pcb-rescue:L-Device-pcb-rescue L401
+L Device:L_Small L401
 U 1 1 5D4971D8
 P 4200 2450
@@
 $EndComp
 $Comp
-L pcb-rescue:L-Device-pcb-rescue L400
+L Device:L_Small L400
 U 1 1 5D4999E2
 P 3500 2450
@@
 $EndComp
 $Comp
-L pcb-rescue:R_POT-Device-pcb-rescue RV?
+L Device:R_POT RV?
 U 1 1 5D1F1382
 P 2400 5900
@@
 $EndComp
 $Comp
-L pcb-rescue:GND-power-pcb-rescue #PWR0275
+L power:GND #PWR0275
 U 1 1 5D1F4706
 P 2400 6200
@@
 $EndComp
 $Comp
-L pcb-rescue:+3V3-power-pcb-rescue #PWR0276
+L power:+3V3 #PWR0276
 U 1 1 5D1F4C5C
 P 2400 5600
@@
 Connection ~ 4900 5700
 $Comp
-L pcb-rescue:AudioJack3_SwitchTR-Connector-pcb-rescue J1
+L Connector:AudioJack3_SwitchTR J1
 U 1 1 5D440F5D
 P 7850 5100
@@
 	6600 5100 7650 5100
 $Comp
-L pcb-rescue:GND-power-pcb-rescue #PWR0165
+L power:GND #PWR0165
 U 1 1 5D462232
 P 7550 5000

Commit message: pcb: bug fixes
Parts:
- L400, L401: symbol Device:L_Small -> Device:L
Connections:
- net +1V8: now also L400.1, L401.1
- net at C401.1, C402.1, U400.31 (VL)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: now also L401.2
- net at C400.1, X400.1 (EN), X400.4 (Vdd): now also L400.2
Changed lines of the file:
@@
 	3800 3500 5000 3500
 $Comp
-L Device:L_Small L401
+L Device:L L401
 U 1 1 5D4971D8
 P 4200 2450
@@
 $EndComp
 $Comp
-L Device:L_Small L400
+L Device:L L400
 U 1 1 5D4999E2
 P 3500 2450
